Commit message: Fixed indentations and formatting issues

File: rox_description/urdf/xacros/argo_drive.xacro (robot description, xacro)
@@ -7,20 +7,20 @@
         vis_rot="0 0 0" vis_pos="0 0 0"
         joint_type="${joint_typ}">
-        <origin rpy="0 0 ${pi}" xyz="${0.239} 0.229 0.123"/>
+        <origin rpy="0 0 ${pi}" xyz="0.239 0.229 0.123"/>
     </xacro:argo_caster>
     <xacro:argo_caster name="caster_front_right" parent="${parent}"
         vis_rot="0 0 ${pi}" vis_pos="0 0 0"
         joint_type="${joint_typ}">
-        <origin rpy="0 0 0" xyz="${0.239} -0.229 0.123"/>
+        <origin rpy="0 0 0" xyz="0.239 -0.229 0.123"/>
     </xacro:argo_caster>
     <xacro:argo_caster name="caster_back_left" parent="${parent}"
         vis_rot="0 0 0" vis_pos="0 0 0"
         joint_type="${joint_typ}">
-        <origin rpy="0 0 ${pi}" xyz="-${0.239} 0.229 0.123"/>
+        <origin rpy="0 0 ${pi}" xyz="-0.239 0.229 0.123"/>
     </xacro:argo_caster>
     <xacro:argo_caster name="caster_back_right" parent="${parent}"
         vis_rot="0 0 ${pi}" vis_pos="0 0 0"
         joint_type="${joint_typ}">
-        <origin rpy="0 0 0" xyz="-${0.239} -0.229 0.123"/>
+        <origin rpy="0 0 0" xyz="-0.239 -0.229 0.123"/>
     </xacro:argo_caster>
     <xacro:argo_wheel name="wheel_front_left" parent="caster_front_left_link"

File: rox_description/urdf/xacros/diff_drive.xacro (robot description, xacro)
@@ -7,5 +7,5 @@
         vis_rot="-${pi/2} 0 ${pi/2}" vis_pos="0 0 0" collision_pos="0.045 0 0"
         joint_type="fixed">
-        <origin rpy="0 0 0" xyz="${0.2045 + 0.045} -0.220 0.124"/>
+        <origin rpy="0 0 0" xyz="0.2495 -0.220 0.124"/>
         <!-- For the caster position 0.2785 is L3.2 and 0.045 is the Swivel lead -->
     </xacro:diff_caster>
@@ -13,5 +13,5 @@
         vis_rot="-${pi/2} 0 ${pi/2}" vis_pos="0 0 0" collision_pos="0.045 0 0"
         joint_type="fixed">
-        <origin rpy="0 0 0" xyz="${0.2045 + 0.045} 0.220 0.124"/>
+        <origin rpy="0 0 0" xyz="0.2495 0.220 0.124"/>
         <!-- For the caster position 0.2785 is L3.2 and 0.045 is the Swivel lead -->
     </xacro:diff_caster>
@@ -19,5 +19,5 @@
         vis_rot="-${pi/2} 0 ${pi/2}" vis_pos="0 0 0" collision_pos="0.045 0 0"
         joint_type="fixed">
-        <origin rpy="0 0 0" xyz="-${0.2945 - 0.045} -0.220 0.124"/>
+        <origin rpy="0 0 0" xyz="-0.1595 -0.220 0.124"/>
         <!-- For the caster position 0.1885 is L3.2 and 0.045 is the Swivel lead -->
     </xacro:diff_caster>
@@ -25,5 +25,5 @@
         vis_rot="-${pi/2} 0 ${pi/2}" vis_pos="0 0 0" collision_pos="0.045 0 0"
         joint_type="fixed">
-        <origin rpy="0 0 0" xyz="-${0.2945 - 0.045} 0.220 0.124"/>
+        <origin rpy="0 0 0" xyz="-0.1595 0.220 0.124"/>
         <!-- For the caster position 0.1885 is L3.2 and 0.045 is the Swivel lead -->
     </xacro:diff_caster>

File: rox_description/urdf/xacros/elite_arm.urdf.xacro (robot description, xacro)
@@ -1,62 +1,59 @@
 <?xml version="1.0"?>
-<!-- This is the main URDF file for mpo_700-->
+<!--
+Author: Pradheep Padmanabhan
+Contributor: Adarsh Karan K P
+-->
 <robot xmlns:xacro="http://www.ros.org/wiki/xacro" name="elite">
-            <!--
-                Author: Adarsh Karan K P
-            -->
-            <!-- Include macros -->
-            <xacro:include filename="$(find elite_description)/urdf/macro/elite_macro.xacro" />
-            <!-- Set use_gz = true for simulation -->
-            <xacro:arg name="use_gz" default="false"/>
-            <!-- arm parameters -->
-            <xacro:arg name="arm_type" default="ec66"/>
-            <xacro:arg name="arm_parent" default="world"/>
-            <!--Elite arm parameters-->
-            <xacro:arg name="tf_prefix" default="$(arg arm_type)" />
-            <xacro:arg name="joint_limit_params_file" default="$(find elite_description)/config/$(arg arm_type)/joint_limits.yaml"/>
-            <xacro:arg name="kinematics_params_file" default="$(find elite_description)/config/$(arg arm_type)/kinematics.yaml"/>
-            <xacro:arg name="physical_params_file" default="$(find elite_description)/config/$(arg arm_type)/physical_parameters.yaml"/>
-            <!-- initial positions file for Elite arm on rox-->
-            <xacro:arg name="initial_joint_positions_file" default="$(find elite_description)/config/$(arg arm_type)/initial_positions.yaml"/>
-            <!-- Load parameters from YAML file -->
-            <xacro:property
-                name="elite_initial_positions"
-                value="${xacro.load_yaml('$(arg initial_joint_positions_file)')}"
-            />
-            <!--create arm from macro-->
-            <xacro:elite_robot
-                name="$(arg arm_type)"
-                tf_prefix="$(arg tf_prefix)"
-                parent="$(arg arm_parent)"
-                joint_limits_parameters_file="$(arg joint_limit_params_file)"
-                kinematics_parameters_file="$(arg kinematics_params_file)"
-                physical_parameters_file="$(arg physical_params_file)"
-                >
-                <origin xyz="0.218 0.0 ${arm_height}" rpy="0.0 0.0 3.1415926535897931" />
-            </xacro:elite_robot>
-            <!-- this condition is to ensure that ros2_control doesn't interfere with gz_ros2_control during simulation  -->
-            <!-- <xacro:unless value="$(arg use_gz)">
-            </xacro:unless> -->
-            <!-- If gz simulation is used -->
-            <xacro:if value="$(arg use_gz)">
-                <xacro:include filename="$(find elite_description)/urdf/macro/elite_ros2_control_macro.xacro" />
-                <xacro:arg name="simulation_controllers" default="$(find rox_bringup)/configs/elite/$(arg arm_type)/elite_controllers.yaml"/>
-                <gazebo reference="$(arg arm_parent)">
-                </gazebo>
-                <gazebo>
-                    <plugin name="gz_ros2_control::GazeboSimROS2ControlPlugin" filename="libgz_ros2_control-system">
-                        <parameters>$(arg simulation_controllers)</parameters>
-                    </plugin>
-                </gazebo>
-                <!-- Use the Elite_ros2_control macro -->
-                <xacro:elite_ros2_control
-                    name="GazeboSimSystem"
-                    tf_prefix="$(arg tf_prefix)"
-                    plugin="gz_ros2_control/GazeboSimSystem"
-                    parameters="$(arg simulation_controllers)"
-                    initial_positions="${elite_initial_positions}"
-                />
-            </xacro:if>
-            <!-- include robotiq gripper-->
-            <!-- <xacro:include filename="$(find neo_simulation2)/components/arm/robotiq_gripper.urdf.xacro"/> -->
+  <!-- Set use_gz = true for simulation -->
+  <xacro:arg name="use_gz" default="false"/>
+  <!-- arm parameters -->
+  <xacro:arg name="arm_type" default="ec66"/>
+  <!-- Include macros -->
+  <xacro:include filename="$(find elite_description)/urdf/xacros/elite_macro.xacro" />
+  <!--Elite arm parameters -->
+  <xacro:arg name="arm_parent" default="world"/>
+  <xacro:arg name="tf_prefix" default="$(arg arm_type)" />
+  <xacro:arg name="joint_limit_params_file" default="$(find elite_description)/config/$(arg arm_type)/joint_limits.yaml"/>
+  <xacro:arg name="kinematics_params_file" default="$(find elite_description)/config/$(arg arm_type)/kinematics.yaml"/>
+  <xacro:arg name="physical_params_file" default="$(find elite_description)/config/$(arg arm_type)/physical_parameters.yaml"/>
+  <!-- initial positions file for Elite arm on rox -->
+  <xacro:arg name="initial_joint_positions_file" default="$(find rox_bringup)/configs/elite/initial_positions.yaml"/>
+  <!-- Load parameters from YAML file -->
+  <xacro:property
+    name="elite_initial_positions"
+    value="${xacro.load_yaml('$(arg initial_joint_positions_file)')}"
+    />
+  <!--create arm from macro -->
+  <xacro:elite_robot
+    name="$(arg arm_type)"
+    tf_prefix="$(arg tf_prefix)"
+    parent="$(arg arm_parent)"
+    joint_limits_parameters_file="$(arg joint_limit_params_file)"
+    kinematics_parameters_file="$(arg kinematics_params_file)"
+    physical_parameters_file="$(arg physical_params_file)"
+    >
+    <origin xyz="0.218 0.0 ${arm_height}" rpy="0.0 0.0 3.1415926535897931" />
+  </xacro:elite_robot>
+  <!-- If gz simulation is used -->
+  <xacro:if value="$(arg use_gz)">
+    <xacro:include filename="$(find elite_description)/urdf/xacros/elite_ros2_control_macro.xacro" />
+    <xacro:arg name="simulation_controllers" default="$(find rox_bringup)/configs/elite/$(arg arm_type)/elite_controllers.yaml"/>
+    <gazebo reference="$(arg arm_parent)">
+    </gazebo>
+    <gazebo>
+      <plugin name="gz_ros2_control::GazeboSimROS2ControlPlugin" filename="libgz_ros2_control-system">
+        <parameters>$(arg simulation_controllers)</parameters>
+      </plugin>
+    </gazebo>
+    <!-- Use the Elite_ros2_control macro -->
+    <xacro:elite_ros2_control
+      name="GazeboSimSystem"
+      tf_prefix="$(arg tf_prefix)"
+      plugin="gz_ros2_control/GazeboSimSystem"
+      parameters="$(arg simulation_controllers)"
+      initial_positions="${elite_initial_positions}"
+      />
+  </xacro:if>
+  <!-- include robotiq gripper-->
+  <!-- <xacro:include filename="$(find neo_simulation2)/components/arm/robotiq_gripper.urdf.xacro"/> -->
 </robot>

File: rox_description/urdf/xacros/trike_drive.xacro (robot description, xacro)
@@ -7,5 +7,5 @@
         vis_rot="-${pi/2} 0 -${pi/2}" vis_pos="0 0 0" collision_pos="-0.045 0 0"
         joint_type="fixed">
-        <origin rpy="0 0 0" xyz="-${0.2785 - 0.045} 0.0 0.124"/>
+        <origin rpy="0 0 0" xyz="-0.2335 0.0 0.124"/>
         <!-- For the caster position 0.2785 is L3.2 and 0.045 is the Swivel lead -->
     </xacro:diff_caster>
