Commit message: Fixed indentations and formatting issues

File: rox_description/urdf/xacros/ur_arm.urdf.xacro (robot description, xacro)
@@ -1,131 +1,130 @@
 <?xml version="1.0"?>
-<!-- This is the main URDF file for mpo_700-->
+<!--
+Author: Pradheep Padmanabhan
+Contributor: Adarsh Karan K P
+-->
 <robot xmlns:xacro="http://www.ros.org/wiki/xacro" name="ur">
-  <!--
-    Author: Pradheep Padmanabhan
-    Contributor: Adarsh Karan K P
-  -->
-            <!-- create arm from macro-->
-            <xacro:include filename="$(find ur_description)/urdf/ur_macro.xacro"/>
-            <xacro:include filename="$(find ur_robot_driver)/urdf/ur.ros2_control.xacro"/>
-            <xacro:include filename="$(find ur_description)/urdf/inc/ur_transmissions.xacro"/>
-            <!-- Set use_gz = true for simulation -->
-            <xacro:arg name="use_gz" default="false"/>
-            <!-- arm parameters -->
-            <xacro:arg name="arm_type" default="ur10"/>
-            <xacro:property name="arm_height" default="0" />
-            <xacro:arg name="arm_parent" default="world"/>
-            <!-- UR arm parameters -->
-            <xacro:arg name="tf_prefix" default="$(arg arm_type)" />
-            <xacro:arg name="joint_limit_params" default="$(find ur_description)/config/$(arg arm_type)/joint_limits.yaml"/>
-            <xacro:arg name="kinematics_params" default="$(find ur_description)/config/$(arg arm_type)/default_kinematics.yaml"/>
-            <xacro:arg name="physical_params" default="$(find ur_description)/config/$(arg arm_type)/physical_parameters.yaml"/>
-            <xacro:arg name="visual_params" default="$(find ur_description)/config/$(arg arm_type)/visual_parameters.yaml"/>
-            <xacro:arg name="transmission_hw_interface" default="hardware_interface/PositionJointInterface"/>
-            <xacro:arg name="safety_limits" default="false"/>
-            <xacro:arg name="safety_pos_margin" default="0.15"/>
-            <xacro:arg name="safety_k_position" default="20"/>
-            <!-- initial positions file for ur arm on rox-->
-            <xacro:arg name="initial_positions_file" default="$(find rox_bringup)/configs/ur/initial_joint_positions.yaml"/>
-            <!-- When using gazebo simulations absolute paths are necessary -->
-            <xacro:arg name="force_abs_paths" default="false" />
-            <!-- parse initial positions as a dictionary -->
-            <xacro:property
-                name="ur_initial_positions"
-                value="${xacro.load_yaml('$(arg initial_positions_file)')}"
-                />
-            <!-- create arm from macro-->
-            <xacro:ur_robot
-                name="$(arg arm_type)"
-                parent="$(arg arm_parent)"
-                tf_prefix="$(arg tf_prefix)"
-                joint_limits_parameters_file="$(arg joint_limit_params)"
-                kinematics_parameters_file="$(arg kinematics_params)"
-                physical_parameters_file="$(arg physical_params)"
-                visual_parameters_file="$(arg visual_params)"
-                safety_limits="$(arg safety_limits)"
-                safety_pos_margin="$(arg safety_pos_margin)"
-                safety_k_position="$(arg safety_k_position)"
-                force_abs_paths="$(arg force_abs_paths)"
-                >
-                <!-- position of arm in the world -->
-                <origin xyz="0.218 0.0 ${arm_height}" rpy="0.0 0.0 3.1415926535897931" />
-            </xacro:ur_robot>
-            <!-- this condition is to ensure that ros2_control doesn't interfere with gz_ros2_control during simulation  -->
-            <xacro:unless value="$(arg use_gz)">
-                <!-- ros2_control related parameters -->
-                <xacro:arg name="headless_mode" default="false" />
-                <xacro:arg name="robot_ip" default="192.168.1.102" />
-                <xacro:arg name="script_filename" default="$(find ur_client_library)/resources/external_control.urscript"/>
-                <xacro:arg name="output_recipe_filename" default="$(find ur_robot_driver)/resources/rtde_output_recipe.txt"/>
-                <xacro:arg name="input_recipe_filename" default="$(find ur_robot_driver)/resources/rtde_input_recipe.txt"/>
-                <xacro:arg name="reverse_ip" default="0.0.0.0"/>
-                <xacro:arg name="script_command_port" default="50004"/>
-                <xacro:arg name="reverse_port" default="50001"/>
-                <xacro:arg name="script_sender_port" default="50002"/>
-                <xacro:arg name="trajectory_port" default="50003"/>
-                <!-- tool communication related parameters-->
-                <xacro:arg name="use_tool_communication" default="false" />
-                <xacro:arg name="tool_voltage" default="0" />
-                <xacro:arg name="tool_parity" default="0" />
-                <xacro:arg name="tool_baud_rate" default="115200" />
-                <xacro:arg name="tool_stop_bits" default="1" />
-                <xacro:arg name="tool_rx_idle_chars" default="1.5" />
-                <xacro:arg name="tool_tx_idle_chars" default="3.5" />
-                <xacro:arg name="tool_device_name" default="/tmp/ttyUR" />
-                <xacro:arg name="tool_tcp_port" default="54321" />
-                <xacro:arg name="use_mock_hardware" default="false" />
-                <xacro:arg name="mock_sensor_commands" default="false" />
-                <xacro:ur_ros2_control
-                    name="$(arg arm_type)"
-                    tf_prefix="$(arg tf_prefix)"
-                    kinematics_parameters_file="$(arg kinematics_params)"
-                    transmission_hw_interface="$(arg transmission_hw_interface)"
-                    headless_mode="$(arg headless_mode)"
-                    initial_positions="${ur_initial_positions}"
-                    use_tool_communication="$(arg use_tool_communication)"
-                    tool_voltage="$(arg tool_voltage)"
-                    tool_parity="$(arg tool_parity)"
-                    tool_baud_rate="$(arg tool_baud_rate)"
-                    tool_stop_bits="$(arg tool_stop_bits)"
-                    tool_rx_idle_chars="$(arg tool_rx_idle_chars)"
-                    tool_tx_idle_chars="$(arg tool_tx_idle_chars)"
-                    tool_device_name="$(arg tool_device_name)"
-                    tool_tcp_port="$(arg tool_tcp_port)"
-                    robot_ip="$(arg robot_ip)"
-                    script_filename="$(arg script_filename)"
-                    output_recipe_filename="$(arg output_recipe_filename)"
-                    input_recipe_filename="$(arg input_recipe_filename)"
-                    reverse_ip="$(arg reverse_ip)"
-                    script_command_port="$(arg script_command_port)"
-                    reverse_port="$(arg reverse_port)"
-                    script_sender_port="$(arg script_sender_port)"
-                    trajectory_port="$(arg trajectory_port)"
-                    use_mock_hardware="$(arg use_mock_hardware)"
-                    mock_sensor_commands="$(arg mock_sensor_commands)"
-                />
-            </xacro:unless>
-            <!-- If gz simulation is used -->
-            <xacro:if value="$(arg use_gz)">
-                <!-- simulation controllers will be passed from launch file after substitutions -->
-                <xacro:arg name="simulation_controllers" default=""/>
-                <gazebo reference="$(arg arm_parent)">
-                </gazebo>
-                <gazebo>
-                    <plugin name="gz_ros2_control::GazeboSimROS2ControlPlugin" filename="libgz_ros2_control-system">
-                        <parameters>$(arg simulation_controllers)</parameters>
-                        <!-- <controller_manager_node_name>$(arg tf_prefix)controller_manager</controller_manager_node_name> -->
-                    </plugin>
-                </gazebo>
-                <!-- ros2 control instance -->
-                <xacro:include filename="$(find ur_simulation_gz)/urdf/ur_gz.ros2_control.xacro" />
-                <xacro:ur_ros2_control
-                    name="$(arg arm_type)"
-                    tf_prefix="$(arg tf_prefix)"
-                    transmission_hw_interface="$(arg transmission_hw_interface)"
-                    initial_positions="${ur_initial_positions}"
-                />
-            </xacro:if>
-            <!-- include robotiq gripper-->
-            <!-- <xacro:include filename="$(find neo_simulation2)/components/arm/robotiq_gripper.urdf.xacro"/> -->
+  <!-- create arm from macro-->
+  <xacro:include filename="$(find ur_description)/urdf/ur_macro.xacro"/>
+  <xacro:include filename="$(find ur_robot_driver)/urdf/ur.ros2_control.xacro"/>
+  <xacro:include filename="$(find ur_description)/urdf/inc/ur_transmissions.xacro"/>
+  <!-- Set use_gz = true for simulation -->
+  <xacro:arg name="use_gz" default="false"/>
+  <!-- arm parameters -->
+  <xacro:arg name="arm_type" default="ur10"/>
+  <xacro:property name="arm_height" default="0" />
+  <xacro:arg name="arm_parent" default="world"/>
+  <!-- UR arm parameters -->
+  <xacro:arg name="tf_prefix" default="$(arg arm_type)" />
+  <xacro:arg name="joint_limit_params" default="$(find ur_description)/config/$(arg arm_type)/joint_limits.yaml"/>
+  <xacro:arg name="kinematics_params" default="$(find ur_description)/config/$(arg arm_type)/default_kinematics.yaml"/>
+  <xacro:arg name="physical_params" default="$(find ur_description)/config/$(arg arm_type)/physical_parameters.yaml"/>
+  <xacro:arg name="visual_params" default="$(find ur_description)/config/$(arg arm_type)/visual_parameters.yaml"/>
+  <xacro:arg name="transmission_hw_interface" default="hardware_interface/PositionJointInterface"/>
+  <xacro:arg name="safety_limits" default="false"/>
+  <xacro:arg name="safety_pos_margin" default="0.15"/>
+  <xacro:arg name="safety_k_position" default="20"/>
+  <!-- initial positions file for ur arm on rox-->
+  <xacro:arg name="initial_positions_file" default="$(find rox_bringup)/configs/ur/initial_joint_positions.yaml"/>
+  <!-- When using gazebo simulations absolute paths are necessary -->
+  <xacro:arg name="force_abs_paths" default="false" />
+  <!-- parse initial positions as a dictionary -->
+  <xacro:property
+    name="ur_initial_positions"
+    value="${xacro.load_yaml('$(arg initial_positions_file)')}"
+    />
+  <!-- create arm from macro-->
+  <xacro:ur_robot
+    name="$(arg arm_type)"
+    parent="$(arg arm_parent)"
+    tf_prefix="$(arg tf_prefix)"
+    joint_limits_parameters_file="$(arg joint_limit_params)"
+    kinematics_parameters_file="$(arg kinematics_params)"
+    physical_parameters_file="$(arg physical_params)"
+    visual_parameters_file="$(arg visual_params)"
+    safety_limits="$(arg safety_limits)"
+    safety_pos_margin="$(arg safety_pos_margin)"
+    safety_k_position="$(arg safety_k_position)"
+    force_abs_paths="$(arg force_abs_paths)"
+    >
+    <!-- position of arm in the world -->
+    <origin xyz="0.218 0.0 ${arm_height}" rpy="0.0 0.0 3.1415926535897931" />
+  </xacro:ur_robot>
+  <!-- this condition is to ensure that ros2_control doesn't interfere with gz_ros2_control during simulation  -->
+  <xacro:unless value="$(arg use_gz)">
+    <!-- ros2_control related parameters -->
+    <xacro:arg name="headless_mode" default="false" />
+    <xacro:arg name="robot_ip" default="192.168.1.102" />
+    <xacro:arg name="script_filename" default="$(find ur_client_library)/resources/external_control.urscript"/>
+    <xacro:arg name="output_recipe_filename" default="$(find ur_robot_driver)/resources/rtde_output_recipe.txt"/>
+    <xacro:arg name="input_recipe_filename" default="$(find ur_robot_driver)/resources/rtde_input_recipe.txt"/>
+    <xacro:arg name="reverse_ip" default="0.0.0.0"/>
+    <xacro:arg name="script_command_port" default="50004"/>
+    <xacro:arg name="reverse_port" default="50001"/>
+    <xacro:arg name="script_sender_port" default="50002"/>
+    <xacro:arg name="trajectory_port" default="50003"/>
+    <!-- tool communication related parameters-->
+    <xacro:arg name="use_tool_communication" default="false" />
+    <xacro:arg name="tool_voltage" default="0" />
+    <xacro:arg name="tool_parity" default="0" />
+    <xacro:arg name="tool_baud_rate" default="115200" />
+    <xacro:arg name="tool_stop_bits" default="1" />
+    <xacro:arg name="tool_rx_idle_chars" default="1.5" />
+    <xacro:arg name="tool_tx_idle_chars" default="3.5" />
+    <xacro:arg name="tool_device_name" default="/tmp/ttyUR" />
+    <xacro:arg name="tool_tcp_port" default="54321" />
+    <xacro:arg name="use_mock_hardware" default="false" />
+    <xacro:arg name="mock_sensor_commands" default="false" />
+    <xacro:ur_ros2_control
+      name="$(arg arm_type)"
+      tf_prefix="$(arg tf_prefix)"
+      kinematics_parameters_file="$(arg kinematics_params)"
+      transmission_hw_interface="$(arg transmission_hw_interface)"
+      headless_mode="$(arg headless_mode)"
+      initial_positions="${ur_initial_positions}"
+      use_tool_communication="$(arg use_tool_communication)"
+      tool_voltage="$(arg tool_voltage)"
+      tool_parity="$(arg tool_parity)"
+      tool_baud_rate="$(arg tool_baud_rate)"
+      tool_stop_bits="$(arg tool_stop_bits)"
+      tool_rx_idle_chars="$(arg tool_rx_idle_chars)"
+      tool_tx_idle_chars="$(arg tool_tx_idle_chars)"
+      tool_device_name="$(arg tool_device_name)"
+      tool_tcp_port="$(arg tool_tcp_port)"
+      robot_ip="$(arg robot_ip)"
+      script_filename="$(arg script_filename)"
+      output_recipe_filename="$(arg output_recipe_filename)"
+      input_recipe_filename="$(arg input_recipe_filename)"
+      reverse_ip="$(arg reverse_ip)"
+      script_command_port="$(arg script_command_port)"
+      reverse_port="$(arg reverse_port)"
+      script_sender_port="$(arg script_sender_port)"
+      trajectory_port="$(arg trajectory_port)"
+      use_mock_hardware="$(arg use_mock_hardware)"
+      mock_sensor_commands="$(arg mock_sensor_commands)"
+      />
+  </xacro:unless>
+  <!-- If gz simulation is used -->
+  <xacro:if value="$(arg use_gz)">
+    <!-- simulation controllers will be passed from launch file after substitutions -->
+    <xacro:arg name="simulation_controllers" default=""/>
+    <gazebo reference="$(arg arm_parent)">
+    </gazebo>
+    <gazebo>
+      <plugin name="gz_ros2_control::GazeboSimROS2ControlPlugin" filename="libgz_ros2_control-system">
+        <parameters>$(arg simulation_controllers)</parameters>
+        <!-- <controller_manager_node_name>$(arg tf_prefix)controller_manager</controller_manager_node_name> -->
+      </plugin>
+    </gazebo>
+    <!-- ros2 control instance -->
+    <xacro:include filename="$(find ur_simulation_gz)/urdf/ur_gz.ros2_control.xacro" />
+    <xacro:ur_ros2_control
+      name="$(arg arm_type)"
+      tf_prefix="$(arg tf_prefix)"
+      transmission_hw_interface="$(arg transmission_hw_interface)"
+      initial_positions="${ur_initial_positions}"
+      />
+  </xacro:if>
+  <!-- include robotiq gripper-->
+  <!-- <xacro:include filename="$(find neo_simulation2)/components/arm/robotiq_gripper.urdf.xacro"/> -->
 </robot>
