Commit message: minor updates to launch files and urdf

File: rox_description/urdf/xacros/elite_arm.urdf.xacro (robot description, xacro)
@@ -21,9 +21,7 @@
             <!-- Load parameters from YAML file -->
             <xacro:property
-                name="initial_positions_params"
+                name="elite_initial_positions"
                 value="${xacro.load_yaml('$(arg initial_joint_positions_file)')}"
             />
-            <!-- Extract subsection from yaml dictionaries -->
-            <xacro:property name="elite_initial_positions" value="${initial_positions_params['initial_positions']}"/>
             <!--create arm from macro-->
             <xacro:elite_robot
@@ -57,4 +55,5 @@
                     plugin="gz_ros2_control/GazeboSimSystem"
                     parameters="$(arg simulation_controllers)"
+                    initial_positions="${elite_initial_positions}"
                 />
             </xacro:if>

File: rox_description/urdf/xacros/ur_arm.urdf.xacro (robot description, xacro)
@@ -8,6 +8,6 @@
             <!-- create arm from macro-->
             <xacro:include filename="$(find ur_description)/urdf/ur_macro.xacro"/>
-            <xacro:include filename="$(find ur_robot_driver)/urdf/ur.ros2_control.xacro" />
-            <xacro:include filename="$(find ur_description)/urdf/inc/ur_transmissions.xacro" />
+            <xacro:include filename="$(find ur_robot_driver)/urdf/ur.ros2_control.xacro"/>
+            <xacro:include filename="$(find ur_description)/urdf/inc/ur_transmissions.xacro"/>
             <!-- Set use_gz = true for simulation -->
             <xacro:arg name="use_gz" default="false"/>
@@ -26,25 +26,4 @@
             <xacro:arg name="safety_pos_margin" default="0.15"/>
             <xacro:arg name="safety_k_position" default="20"/>
-            <!-- ros2_control related parameters -->
-            <xacro:arg name="headless_mode" default="false" />
-            <xacro:arg name="robot_ip" default="192.168.1.102" />
-            <xacro:arg name="script_filename" default="$(find ur_client_library)/resources/external_control.urscript"/>
-            <xacro:arg name="output_recipe_filename" default="$(find ur_robot_driver)/resources/rtde_output_recipe.txt"/>
-            <xacro:arg name="input_recipe_filename" default="$(find ur_robot_driver)/resources/rtde_input_recipe.txt"/>
-            <xacro:arg name="reverse_ip" default="0.0.0.0"/>
-            <xacro:arg name="script_command_port" default="50004"/>
-            <xacro:arg name="reverse_port" default="50001"/>
-            <xacro:arg name="script_sender_port" default="50002"/>
-            <xacro:arg name="trajectory_port" default="50003"/>
-            <!-- tool communication related parameters-->
-            <xacro:arg name="use_tool_communication" default="false" />
-            <xacro:arg name="tool_voltage" default="0" />
-            <xacro:arg name="tool_parity" default="0" />
-            <xacro:arg name="tool_baud_rate" default="115200" />
-            <xacro:arg name="tool_stop_bits" default="1" />
-            <xacro:arg name="tool_rx_idle_chars" default="1.5" />
-            <xacro:arg name="tool_tx_idle_chars" default="3.5" />
-            <xacro:arg name="tool_device_name" default="/tmp/ttyUR" />
-            <xacro:arg name="tool_tcp_port" default="54321" />
             <!-- initial positions file for ur arm on rox-->
             <xacro:arg name="initial_positions_file" default="$(find rox_bringup)/configs/ur/initial_joint_positions.yaml"/>
@@ -75,4 +54,25 @@
             <!-- this condition is to ensure that ros2_control doesn't interfere with gz_ros2_control during simulation  -->
             <xacro:unless value="$(arg use_gz)">
+                <!-- ros2_control related parameters -->
+                <xacro:arg name="headless_mode" default="false" />
+                <xacro:arg name="robot_ip" default="192.168.1.102" />
+                <xacro:arg name="script_filename" default="$(find ur_client_library)/resources/external_control.urscript"/>
+                <xacro:arg name="output_recipe_filename" default="$(find ur_robot_driver)/resources/rtde_output_recipe.txt"/>
+                <xacro:arg name="input_recipe_filename" default="$(find ur_robot_driver)/resources/rtde_input_recipe.txt"/>
+                <xacro:arg name="reverse_ip" default="0.0.0.0"/>
+                <xacro:arg name="script_command_port" default="50004"/>
+                <xacro:arg name="reverse_port" default="50001"/>
+                <xacro:arg name="script_sender_port" default="50002"/>
+                <xacro:arg name="trajectory_port" default="50003"/>
+                <!-- tool communication related parameters-->
+                <xacro:arg name="use_tool_communication" default="false" />
+                <xacro:arg name="tool_voltage" default="0" />
+                <xacro:arg name="tool_parity" default="0" />
+                <xacro:arg name="tool_baud_rate" default="115200" />
+                <xacro:arg name="tool_stop_bits" default="1" />
+                <xacro:arg name="tool_rx_idle_chars" default="1.5" />
+                <xacro:arg name="tool_tx_idle_chars" default="3.5" />
+                <xacro:arg name="tool_device_name" default="/tmp/ttyUR" />
+                <xacro:arg name="tool_tcp_port" default="54321" />
                 <xacro:ur_ros2_control
                     name="$(arg arm_type)"

Commit message: Changed hardcoded robot_ip value to launch arg value, minor formatting and default value fixes to urdf (#75)

File: rox_description/urdf/xacros/elite_arm.urdf.xacro (robot description, xacro)
@@ -9,4 +9,5 @@
   <!-- arm parameters -->
   <xacro:arg name="arm_type" default="ec66"/>
+  <xacro:property name="arm_height" default="0.376" />
   <!-- Include macros -->
   <xacro:include filename="$(find elite_description)/urdf/xacros/elite_macro.xacro" />

File: rox_description/urdf/xacros/ur_arm.urdf.xacro (robot description, xacro)
@@ -14,5 +14,5 @@
   <!-- arm parameters -->
   <xacro:arg name="arm_type" default="ur10"/>
-  <xacro:property name="arm_height" default="0" />
+  <xacro:property name="arm_height" default="0.376" />
   <xacro:arg name="arm_parent" default="world"/>
   <!-- UR arm parameters -->
