Commit message: Fixed issues with rox argo, diff and trike drive in simulation

File: rox_description/urdf/rox.urdf.xacro (robot description, xacro)
@@ -56,11 +56,12 @@
     <xacro:if value="${rox_typ == 'diff'}">
         <xacro:include filename="$(find rox_description)/urdf/xacros/diff_drive.xacro" />
-        <xacro:diff_drive parent="base_link"/>
+        <xacro:property name="wheel_separation" value="0.634" />
+        <xacro:diff_drive parent="base_link" wheel_separation="${wheel_separation}"/>
     </xacro:if>
     <!-- Trike drive -->
     <xacro:if value="${rox_typ == 'trike'}">
         <xacro:include filename="$(find rox_description)/urdf/xacros/trike_drive.xacro" />
-        <xacro:trike_drive parent="base_link"/>
-        <xacro:property name="frame_len" value="-0.2435" />
+        <xacro:property name="wheel_separation" value="0.5955" />
+        <xacro:trike_drive parent="base_link" wheel_separation="${wheel_separation}"/>
     </xacro:if>
     <!-- Sensors -->

File: rox_description/urdf/xacros/argo_caster.xacro (robot description, xacro)
@@ -5,4 +5,6 @@
     <xacro:insert_block name="origin" />
     <axis xyz="1 0 0" />
+    <joint_properties damping="1." friction="1.0"/>
+    <limit effort="1000.0" lower="-1e+16" upper="1e+16" velocity="100"/>
     <parent link="${parent}" />
     <child link="${name}_link" />
@@ -11,7 +13,7 @@
     <inertial>
     <!-- These are not accurate value -->
-      <mass value="0.025" />
+      <mass value="1.4" />
       <origin xyz="${vis_pos}" rpy="${vis_rot}" />
-      <inertia ixx="0.02" ixy="0" ixz="0" iyy="0.0" iyz="0" izz="0.02" />
+      <inertia ixx="0.00499743171" ixy="0.00000004464" ixz="-0.00000002245" iyy="0.00499741733" iyz="-0.00000000164" izz="0.00839239692"/>
     </inertial>
     <visual>

File: rox_description/urdf/xacros/argo_wheel.xacro (robot description, xacro)
@@ -4,4 +4,6 @@
    <joint name="${name}_joint" type="${joint_type}">
     <xacro:insert_block name="origin" />
+    <limit effort="1000.0" lower="-1e+16" upper="1e+16" velocity="100"/>
+    <joint_properties damping="1.0" friction="1"/>
     <axis xyz="1 0 0" />
     <parent link="${parent}" />
@@ -11,7 +13,7 @@
     <inertial>
     <!-- These are not accurate value -->
-      <mass value="5" />
+      <mass value="1.2" />
       <origin xyz="0 0 0" rpy="0 0 0"/>
-      <inertia ixx="0.02" ixy="0" ixz="0" iyy="0.02" iyz="0" izz="0.02" />
+    <inertia ixx="0.11042056" ixy="0.0" ixz="0.0" iyy="0.11042056" iyz="0.0" izz="0.11042056"/>
     </inertial>
     <visual>

File: rox_description/urdf/xacros/cabinet.xacro (robot description, xacro)
@@ -16,5 +16,5 @@
     <link name="${name}_link">
       <inertial>
-        <mass value="2" />
+        <mass value="10" />
         <origin xyz="0 0 0" rpy="0 0 0"/>
         <inertia ixx="0.457072" ixy="0.0" ixz="0.0"

File: rox_description/urdf/xacros/diff_caster.xacro (robot description, xacro)
@@ -1,7 +1,9 @@
 <?xml version="1.0"?>
 <robot xmlns:xacro="http://www.ros.org/wiki/xacro" name="rox">
-  <xacro:macro name="diff_caster" params="name parent *origin vis_rot vis_pos joint_type">
-    <joint name="${name}_joint" type="fixed">
+  <xacro:macro name="diff_caster" params="name parent *origin vis_rot vis_pos joint_type collision_pos">
+    <joint name="${name}_joint" type="${joint_type}">
       <xacro:insert_block name="origin" />
+      <joint_properties damping="1." friction="1.0"/>
+      <limit effort="1000.0" lower="-1e+16" upper="1e+16" velocity="100"/>
       <axis xyz="1 0 0" />
       <parent link="${parent}" />
@@ -11,9 +13,9 @@
       <inertial>
         <!-- These are not accurate value -->
-        <mass value="0.5" />
+        <mass value="1.4" />
         <origin xyz="${vis_pos}" rpy="${vis_rot}" />
-        <inertia ixx="0.02" ixy="0" ixz="0" iyy="0.02" iyz="0" izz="0.02" />
-      </inertial>
-      <visual>
+        <inertia ixx="0.002" ixy="0" ixz="0" iyy="0.002" iyz="0" izz="0.002" />
+        </inertial>
+        <visual>
         <origin xyz="${vis_pos}" rpy="${vis_rot}" />
         <geometry>
@@ -22,5 +24,5 @@
       </visual>
       <collision>
-        <origin xyz="${vis_pos}" rpy="${vis_rot}" />
+        <origin xyz="${collision_pos}" rpy="${vis_rot}" />
         <geometry>
           <sphere radius="0.124" />

File: rox_description/urdf/xacros/diff_drive.xacro (robot description, xacro)
@@ -3,27 +3,27 @@
   <xacro:include filename="$(find rox_description)/urdf/xacros/diff_caster.xacro" />
   <xacro:include filename="$(find rox_description)/urdf/xacros/diff_wheel.xacro" />
-  <xacro:macro name="diff_drive" params="parent">
-    <xacro:diff_caster name="caster_wheel_front_left" parent="${parent}"
-        vis_rot="-${pi/2} 0 -${pi/2}" vis_pos="0 0 0"
+  <xacro:macro name="diff_drive" params="parent wheel_separation">
+    <xacro:diff_caster name="caster_wheel_front_right" parent="${parent}"
+        vis_rot="-${pi/2} 0 ${pi/2}" vis_pos="0 0 0" collision_pos="0.045 0 0"
         joint_type="fixed">
-        <origin rpy="0 0 0" xyz="${0.2945 + frame_len + 0.045} -0.226 0.124"/>
+        <origin rpy="0 0 0" xyz="${0.2045 + frame_len + 0.045} -0.220 0.124"/>
         <!-- For the caster position 0.2785 is L3.2 and 0.045 is the Swivel lead -->
     </xacro:diff_caster>
-    <xacro:diff_caster name="caster_wheel_front_right" parent="${parent}"
-        vis_rot="-${pi/2} 0 -${pi/2}" vis_pos="0 0 0"
+    <xacro:diff_caster name="caster_wheel_front_left" parent="${parent}"
+        vis_rot="-${pi/2} 0 ${pi/2}" vis_pos="0 0 0" collision_pos="0.045 0 0"
         joint_type="fixed">
-        <origin rpy="0 0 0" xyz="${0.2945 + frame_len + 0.045} 0.226 0.124"/>
+        <origin rpy="0 0 0" xyz="${0.2045 + frame_len + 0.045} 0.220 0.124"/>
         <!-- For the caster position 0.2785 is L3.2 and 0.045 is the Swivel lead -->
     </xacro:diff_caster>
-    <xacro:diff_caster name="caster_wheel_back_left" parent="${parent}"
-        vis_rot="-${pi/2} 0 -${pi/2}" vis_pos="0 0 0"
+    <xacro:diff_caster name="caster_wheel_back_right" parent="${parent}"
+        vis_rot="-${pi/2} 0 ${pi/2}" vis_pos="0 0 0" collision_pos="0.045 0 0"
         joint_type="fixed">
-        <origin rpy="0 0 0" xyz="-${0.2045 + frame_len + 0.045} -0.226 0.124"/>
+        <origin rpy="0 0 0" xyz="-${0.2945 + frame_len - 0.045} -0.220 0.124"/>
         <!-- For the caster position 0.1885 is L3.2 and 0.045 is the Swivel lead -->
     </xacro:diff_caster>
-    <xacro:diff_caster name="caster_wheel_back_right" parent="${parent}"
-        vis_rot="-${pi/2} 0 -${pi/2}" vis_pos="0 0 0"
+    <xacro:diff_caster name="caster_wheel_back_left" parent="${parent}"
+        vis_rot="-${pi/2} 0 ${pi/2}" vis_pos="0 0 0" collision_pos="0.045 0 0"
         joint_type="fixed">
-        <origin rpy="0 0 0" xyz="-${0.2045 + frame_len + 0.045} 0.226 0.124"/>
+        <origin rpy="0 0 0" xyz="-${0.2945 + frame_len - 0.045} 0.220 0.124"/>
         <!-- For the caster position 0.1885 is L3.2 and 0.045 is the Swivel lead -->
     </xacro:diff_caster>
@@ -31,12 +31,10 @@
         vis_rot="0 0 0" vis_pos="0 0 0"
         joint_type="${joint_typ}">
-        <origin xyz="0.0 0.317 0.075" rpy="-${pi/2} 0 0" />
-        <axis xyz="0 0 1" />
+        <origin xyz="0.0 ${wheel_separation/2} 0.075" rpy="0 0 0" />
     </xacro:diff_wheel>
     <xacro:diff_wheel name="wheel_right" parent="${parent}"
         vis_rot="0 ${pi} 0" vis_pos="0 0 0"
         joint_type="${joint_typ}">
-        <origin xyz="0.0 -0.317 0.075" rpy="-${pi/2} 0 0" />
-        <axis xyz="0 0 1" />
+        <origin xyz="0.0 -${wheel_separation/2} 0.075" rpy="0 0 0" />
     </xacro:diff_wheel>
   </xacro:macro>

File: rox_description/urdf/xacros/diff_wheel.xacro (robot description, xacro)
@@ -1,21 +1,21 @@
 <?xml version="1.0"?>
 <robot xmlns:xacro="http://www.ros.org/wiki/xacro" name="rox">
-  <xacro:macro name="diff_wheel" params="name parent vis_rot vis_pos *origin *axis joint_type">
+  <xacro:macro name="diff_wheel" params="name parent vis_rot vis_pos *origin joint_type">
     <joint name="${name}_joint" type="${joint_type}">
       <xacro:insert_block name="origin" />
-      <xacro:insert_block name="axis" />
-      <limit effort="1000.0" lower="-1e+16" upper="1e+16" velocity="100"/>
+    <limit effort="1000.0" lower="-1e+16" upper="1e+16" velocity="100"/>
+    <joint_properties damping="1.0" friction="1"/>
+      <axis xyz="0 1 0" />
       <parent link="${parent}" />
       <child link="${name}_link" />
     </joint>
-    <link name="${name}_link">
+    <link name="${name}_link" type="wheel">
       <inertial>
       <!-- These are not accurate value -->
         <mass value="5.0" />
         <origin xyz="0 0 0" rpy="0 0 0" />
-        <inertia ixx="0.02888" ixy="0" ixz="0" iyy="0.02888" iyz="0" izz="0.05625" />
-      </inertial>
+<inertia ixx="0.02888" ixy="0" ixz="0" iyy="0.02888" iyz="0" izz="0.05625" />      </inertial>
       <visual>
-        <origin xyz="${vis_pos}" rpy="${vis_rot}" />
+        <origin rpy="${pi/2} 0 0" xyz="0 0 0" />
         <geometry>
         <mesh filename="package://rox_description/meshes/diff_wheel.dae" scale="0.001 0.001 0.001"/>
@@ -23,5 +23,5 @@
       </visual>
       <collision>
-        <origin xyz="${vis_pos}" rpy="${vis_rot}" />
+        <origin rpy="0 0 0" xyz="0 0 0" />
         <geometry>
           <sphere radius="0.075" />

File: rox_description/urdf/xacros/frame.xacro (robot description, xacro)
@@ -11,9 +11,7 @@
       <inertial>
       <!-- These are not accurate value -->
-        <mass value="8.0" />
+        <mass value="140.0" />
         <origin xyz="0.0 0 0.18" rpy="0.0 0.0 0.0"/>
-        <inertia ixx="0.299" ixy="0.0" ixz="0.0"
-                 iyy="0.351" iyz="0.0"
-                 izz="0.360" />
+        <inertia ixx="7.8" ixy="0.0" ixz="0" iyy="7.8" iyz="0.0" izz="7.8"/>
       </inertial>
       <visual>

File: rox_description/urdf/xacros/gazebo.xacro (robot description, xacro)
@@ -108,5 +108,5 @@
           <left_joint>wheel_left_joint</left_joint>
           <right_joint>wheel_right_joint</right_joint>
-          <wheel_separation>0.555</wheel_separation>
+          <wheel_separation>${wheel_separation}</wheel_separation>
           <wheel_radius>0.075</wheel_radius>
           <max_linear_acceleration>1</max_linear_acceleration>
@@ -136,4 +136,55 @@
       </plugin>
     </gazebo>
+    <!-- Gazebo macro for Argo Wheels -->
+    <xacro:macro name="rox_argo_wheel_gazebo_macro" params="name">
+      <gazebo reference="${name}_link">
+        <mu1>0.001</mu1>
+        <mu2>0.001</mu2>
+        <kp>100000.0</kp>
+        <kd>1.0</kd>
+        <minDepth>0.000</minDepth>
+        <fdir1>1 0 0</fdir1>
+      </gazebo>
+    </xacro:macro>
+    <!-- Gazebo macro for Differential Castor Wheels -->
+    <xacro:macro name="rox_caster_wheel_gazebo_macro" params="name">
+      <gazebo reference="${name}_link">
+        <mu1>0.001</mu1>
+        <mu2>0.001</mu2>
+      </gazebo>
+    </xacro:macro>
+    <!-- Gazebo macro for Differential Wheels -->
+    <xacro:macro name="rox_diff_wheel_gazebo_macro" params="name">
+      <gazebo reference="${name}_link">
+        <mu1>1.0</mu1>
+        <mu2>1.0</mu2>
+        <kp>1000000.0</kp>
+        <kd>1.0</kd>
+        <minDepth>0.000</minDepth>
+        <fdir1>1 0 0</fdir1>
+      </gazebo>
+    </xacro:macro>
+    <!--Argo Drive-->
+    <xacro:if value="${rox_typ == 'argo'}">
+      <xacro:rox_argo_wheel_gazebo_macro name="wheel_front_left"/>
+      <xacro:rox_argo_wheel_gazebo_macro name="wheel_front_right"/>
+      <xacro:rox_argo_wheel_gazebo_macro name="wheel_back_left"/>
+      <xacro:rox_argo_wheel_gazebo_macro name="wheel_back_right"/>
+    </xacro:if>
+    <!--Diff Drive-->
+    <xacro:if value="${rox_typ == 'diff'}">
+      <xacro:rox_diff_wheel_gazebo_macro name="wheel_left"/>
+      <xacro:rox_diff_wheel_gazebo_macro name="wheel_right"/>
+      <xacro:rox_caster_wheel_gazebo_macro name="caster_wheel_front_left"/>
+      <xacro:rox_caster_wheel_gazebo_macro name="caster_wheel_front_right"/>
+      <xacro:rox_caster_wheel_gazebo_macro name="caster_wheel_back_left"/>
+      <xacro:rox_caster_wheel_gazebo_macro name="caster_wheel_back_right"/>
+    </xacro:if>
+    <!--Trike Drive-->
+    <xacro:if value="${rox_typ == 'trike'}">
+      <xacro:rox_diff_wheel_gazebo_macro name="wheel_left"/>
+      <xacro:rox_diff_wheel_gazebo_macro name="wheel_right"/>
+      <xacro:rox_caster_wheel_gazebo_macro name="caster_back"/>
+    </xacro:if>
   </xacro:macro>
 </robot>

File: rox_description/urdf/xacros/trike_drive.xacro (robot description, xacro)
@@ -3,8 +3,8 @@
   <xacro:include filename="$(find rox_description)/urdf/xacros/diff_caster.xacro" />
   <xacro:include filename="$(find rox_description)/urdf/xacros/diff_wheel.xacro" />
-  <xacro:macro name="trike_drive" params="parent">
+  <xacro:macro name="trike_drive" params="parent wheel_separation">
     <xacro:diff_caster name="caster_back" parent="${parent}"
-        vis_rot="-${pi/2} 0 -${pi/2}" vis_pos="-0.2435 0 0"
-        joint_type="${joint_typ}">
+        vis_rot="-${pi/2} 0 -${pi/2}" vis_pos="0 0 0" collision_pos="-0.045 0 0"
+        joint_type="fixed">
         <origin rpy="0 0 0" xyz="-${0.2785 - 0.045 + frame_len} 0.0 0.124"/>
         <!-- For the caster position 0.2785 is L3.2 and 0.045 is the Swivel lead -->
@@ -13,12 +13,10 @@
         vis_rot="0 0 0" vis_pos="0 0 0"
         joint_type="${joint_typ}">
-        <origin xyz="0.0 0.297 0.075" rpy="-${pi/2} 0 0" />
-        <axis xyz="0 0 1" />
+        <origin xyz="0.2435 ${wheel_separation/2} 0.075" rpy="0 0 0" />
     </xacro:diff_wheel>
     <xacro:diff_wheel name="wheel_right" parent="${parent}"
         vis_rot="0 ${pi} 0" vis_pos="0 0 0"
         joint_type="${joint_typ}">
-        <origin xyz="0.0 -0.297 0.075" rpy="-${pi/2} 0 0" />
-        <axis xyz="0 0 1" />
+        <origin xyz="0.2435 -${wheel_separation/2} 0.075" rpy="0 0 0" />
     </xacro:diff_wheel>
   </xacro:macro>
