Commit message: Updates to Rolling- Migration to Modern Gazebo and addressing Issue 48 (#49)
* Migrate to Modern Gazebo & Modularize URDF for UR & Elite Arms

* Added UR and Elite xacros and controller files

* Updated README.md and added contributor

* Fixed issues with rox argo, diff and trike drive in simulation

* fixes and removing elite desc

* removing the cyclic dependency

---------

Co-authored-by: Pradheep <padhupradheep@gmail.com>

File: rox_description/urdf/rox.urdf.xacro (robot description, xacro)
@@ -11,4 +11,6 @@
     <xacro:arg name="use_d435" default="false"/>
     <xacro:arg name="use_ur_dc" default="false"/>
+    <xacro:arg name="arm_parent" default="cabinet_link"/>
+    <xacro:arg name="force_abs_paths" default="false"/>
     <!-- Xacro Properties -->
     <xacro:property name="frame" value="$(arg frame_type)"/>
@@ -18,5 +20,5 @@
     <xacro:property name="arm" value="$(arg arm_type)"/>
     <xacro:property name="gz" value="$(arg use_gz)"/>
-    <xacro:property name="use_ur_arm" value="false"/>
+    <xacro:property name="use_arm" value="false"/>
     <xacro:property name="imu" value="$(arg use_imu)"/>
     <xacro:property name="d435" value="$(arg use_d435)"/>
@@ -29,6 +31,6 @@
     <xacro:include filename="$(find rox_description)/urdf/xacros/pilz_psenscan.xacro" />
     <!-- checking if one of the UR arms is used -->
-    <xacro:if value="${arm == 'ur5' or arm == 'ur10' or arm == 'ur5e' or arm == 'ur10e'}">
-        <xacro:property name="use_ur_arm" value="true"/>
+    <xacro:if value="${arm == 'ur5' or arm == 'ur10' or arm == 'ur5e' or arm == 'ur10e' or arm == 'ec66' or arm == 'cs66'}">
+        <xacro:property name="use_arm" value="true"/>
     </xacro:if>
     <!-- Assigning Xacro properties -->
@@ -54,11 +56,12 @@
     <xacro:if value="${rox_typ == 'diff'}">
         <xacro:include filename="$(find rox_description)/urdf/xacros/diff_drive.xacro" />
-        <xacro:diff_drive parent="base_link"/>
+        <xacro:property name="wheel_separation" value="0.634" />
+        <xacro:diff_drive parent="base_link" wheel_separation="${wheel_separation}"/>
     </xacro:if>
     <!-- Trike drive -->
     <xacro:if value="${rox_typ == 'trike'}">
         <xacro:include filename="$(find rox_description)/urdf/xacros/trike_drive.xacro" />
-        <xacro:trike_drive parent="base_link"/>
-        <xacro:property name="frame_len" value="-0.2435" />
+        <xacro:property name="wheel_separation" value="0.5955" />
+        <xacro:trike_drive parent="base_link" wheel_separation="${wheel_separation}"/>
     </xacro:if>
     <!-- Sensors -->
@@ -106,94 +109,27 @@
     </xacro:if>
     <!-- arm -->
-    <xacro:unless value="${arm == ''}">
-        <xacro:if value="${ur_dc == False}">
-            <xacro:property name="arm_height" value="0.46" />
-        </xacro:if>
-        <xacro:if value="${ur_dc == True}">
-            <xacro:property name="arm_height" value="0.276" />
-        </xacro:if>
+    <xacro:if value="${use_arm}">
+        <!-- include cabinet -->
         <xacro:include filename="$(find rox_description)/urdf/xacros/cabinet.xacro" />
         <xacro:cabinet name="cabinet" parent="base_footprint">
             <origin rpy="0 0 0" xyz="${frame_len} 0 0.33"/>
         </xacro:cabinet>
-        <xacro:if value="${use_ur_arm == True}">
-            <xacro:include filename="$(find ur_description)/urdf/ur_macro.xacro"/>
-            <xacro:include filename="$(find ur_robot_driver)/urdf/ur.ros2_control.xacro" />
-            <xacro:include filename="$(find ur_description)/urdf/inc/ur_transmissions.xacro" />
-            <xacro:arg name="tf_prefix" default="${arm}" />
-            <xacro:arg name="joint_limit_params" default="$(find ur_description)/config/$(arg arm_type)/joint_limits.yaml"/>
-            <xacro:arg name="kinematics_params" default="$(find ur_description)/config/$(arg arm_type)/default_kinematics.yaml"/>
-            <xacro:arg name="physical_params" default="$(find ur_description)/config/$(arg arm_type)/physical_parameters.yaml"/>
-            <xacro:arg name="visual_params" default="$(find ur_description)/config/$(arg arm_type)/visual_parameters.yaml"/>
-            <xacro:arg name="initial_positions_file" default="$(find ur_description)/config/initial_positions.yaml"/>
-            <xacro:arg name="transmission_hw_interface" default="hardware_interface/PositionJointInterface"/>
-            <xacro:arg name="safety_limits" default="true"/>
-            <xacro:arg name="safety_pos_margin" default="0.15"/>
-            <xacro:arg name="safety_k_position" default="20"/>
-            <xacro:arg name="force_abs_paths" default="false" />
-            <!-- ros2_control related parameters -->
-            <xacro:arg name="headless_mode" default="false" />
-            <xacro:arg name="robot_ip" default="192.168.1.102" />
-            <xacro:arg name="script_filename" default="$(find ur_client_library)/resources/external_control.urscript"/>
-            <xacro:arg name="output_recipe_filename" default="$(find ur_robot_driver)/resources/rtde_output_recipe.txt"/>
-            <xacro:arg name="input_recipe_filename" default="$(find ur_robot_driver)/resources/rtde_input_recipe.txt"/>
-            <xacro:arg name="reverse_ip" default="0.0.0.0"/>
-            <xacro:arg name="script_command_port" default="50004"/>
-            <xacro:arg name="reverse_port" default="50001"/>
-            <xacro:arg name="script_sender_port" default="50002"/>
-            <xacro:arg name="trajectory_port" default="50003"/>
-            <!--   tool communication related parameters-->
-            <xacro:arg name="use_tool_communication" default="false" />
-            <xacro:arg name="tool_voltage" default="0" />
-            <xacro:arg name="tool_parity" default="0" />
-            <xacro:arg name="tool_baud_rate" default="115200" />
-            <xacro:arg name="tool_stop_bits" default="1" />
-            <xacro:arg name="tool_rx_idle_chars" default="1.5" />
-            <xacro:arg name="tool_tx_idle_chars" default="3.5" />
-            <xacro:arg name="tool_device_name" default="/tmp/ttyUR" />
-            <xacro:arg name="tool_tcp_port" default="54321" />
-            <xacro:property name="initial_positions_file" default="$(arg initial_positions_file)"/>
-            <xacro:ur_robot name="${arm}"
-                parent="cabinet_link"
-                tf_prefix="$(arg tf_prefix)"
-                joint_limits_parameters_file="$(arg joint_limit_params)"
-                kinematics_parameters_file="$(arg kinematics_params)"
-                physical_parameters_file="$(arg physical_params)"
-                visual_parameters_file="$(arg visual_params)"
-                safety_limits="$(arg safety_limits)"
-                safety_pos_margin="$(arg safety_pos_margin)"
-                safety_k_position="$(arg safety_k_position)"
-                >
-                <!-- position robot in the world -->
-                <origin xyz="0.218 0.0 ${arm_height}" rpy="0.0 0.0 3.1415926535897931" />
-            </xacro:ur_robot>
-            <xacro:ur_ros2_control
-                name="ur10e"
-                tf_prefix="$(arg tf_prefix)"
-                kinematics_parameters_file="$(arg kinematics_params)"
-                transmission_hw_interface="$(arg transmission_hw_interface)"
-                headless_mode="$(arg headless_mode)"
-                initial_positions="${xacro.load_yaml(initial_positions_file)}"
-                use_tool_communication="$(arg use_tool_communication)"
-                tool_voltage="$(arg tool_voltage)"
-                tool_parity="$(arg tool_parity)"
-                tool_baud_rate="$(arg tool_baud_rate)"
-                tool_stop_bits="$(arg tool_stop_bits)"
-                tool_rx_idle_chars="$(arg tool_rx_idle_chars)"
-                tool_tx_idle_chars="$(arg tool_tx_idle_chars)"
-                tool_device_name="$(arg tool_device_name)"
-                tool_tcp_port="$(arg tool_tcp_port)"
-                robot_ip="$(arg robot_ip)"
-                script_filename="$(arg script_filename)"
-                output_recipe_filename="$(arg output_recipe_filename)"
-                input_recipe_filename="$(arg input_recipe_filename)"
-                reverse_ip="$(arg reverse_ip)"
-                script_command_port="$(arg script_command_port)"
-                reverse_port="$(arg reverse_port)"
-                script_sender_port="$(arg script_sender_port)"
-                trajectory_port="$(arg trajectory_port)"
-            />
+        <!-- Universal Robotics (UR) Arms-->
+        <xacro:if value="${arm == 'ur5' or arm == 'ur10' or arm == 'ur5e' or arm == 'ur10e'}">
+            <xacro:if value="${ur_dc == False}">
+                <!-- Different height for AC arm-->
+                <xacro:property name="arm_height" value="0.376" />
+            </xacro:if>
+            <xacro:if value="${ur_dc == True}">
+                <xacro:property name="arm_height" value="0.276" />
+            </xacro:if>
+            <xacro:include filename="$(find rox_description)/urdf/xacros/ur_arm.urdf.xacro"/>
         </xacro:if>
-    </xacro:unless>
+        <!-- Elite Arms-->
+        <xacro:if value="${arm == 'ec66' or arm == 'cs66'}">
+            <xacro:property name="arm_height" value="0.376" />
+            <xacro:include filename="$(find rox_description)/urdf/xacros/elite_arm.urdf.xacro"/>
+        </xacro:if>
+    </xacro:if>
     <!-- Check if simulation needs to be used -->
     <xacro:if value="${gz == True}">

File: rox_description/urdf/xacros/cabinet.xacro (robot description, xacro)
@@ -3,8 +3,8 @@
   <xacro:macro name="cabinet" params="name parent *origin">
     <joint name="${name}_joint" type="fixed">
-    <xacro:insert_block name="origin" />
-    <joint_properties damping="1" friction="1" />
-    <parent link="${parent}" />
-    <child link="${name}_link" />
+      <xacro:insert_block name="origin" />
+      <joint_properties damping="1" friction="1" />
+      <parent link="${parent}" />
+      <child link="${name}_link" />
     </joint>
     <xacro:if value="${ur_dc == True}">
@@ -16,5 +16,5 @@
     <link name="${name}_link">
       <inertial>
-        <mass value="2" />
+        <mass value="10" />
         <origin xyz="0 0 0" rpy="0 0 0"/>
         <inertia ixx="0.457072" ixy="0.0" ixz="0.0"

File: rox_description/urdf/xacros/gazebo.xacro (robot description, xacro)
@@ -8,5 +8,9 @@
         <visualize>false</visualize>
         <update_rate>10</update_rate>
-        <ray>
+        <topic>scan</topic>
+        <!-- Set output to sensor_msgs/LaserScan to get same output type as gazebo_ros_laser -->
+        <output_type>sensor_msgs/LaserScan</output_type>
+        <gz_frame_id>lidar_1_link</gz_frame_id>
+        <lidar>
           <scan>
             <horizontal>
@@ -31,9 +35,5 @@
             <stddev>0.01</stddev>
           </noise>
-        </ray>
-        <topic>scan</topic>
-        <!-- Set output to sensor_msgs/LaserScan to get same output type as gazebo_ros_laser -->
-        <output_type>sensor_msgs/LaserScan</output_type>
-        <gz_frame_id>lidar_1_link</gz_frame_id>
+        </lidar>
       </sensor>
     </gazebo>
@@ -44,5 +44,9 @@
         <visualize>false</visualize>
         <update_rate>10</update_rate>
-        <ray>
+        <topic>scan2</topic>
+        <!-- Set output to sensor_msgs/LaserScan to get same output type as gazebo_ros_laser -->
+        <output_type>sensor_msgs/LaserScan</output_type>
+        <gz_frame_id>lidar_2_link</gz_frame_id>
+        <lidar>
           <scan>
             <horizontal>
@@ -67,9 +71,5 @@
             <stddev>0.01</stddev>
           </noise>
-        </ray>
-        <topic>scan2</topic>
-        <!-- Set output to sensor_msgs/LaserScan to get same output type as gazebo_ros_laser -->
-        <output_type>sensor_msgs/LaserScan</output_type>
-        <gz_frame_id>lidar_2_link</gz_frame_id>
+        </lidar>
       </sensor>
     </gazebo>
@@ -108,5 +108,5 @@
           <left_joint>wheel_left_joint</left_joint>
           <right_joint>wheel_right_joint</right_joint>
-          <wheel_separation>0.555</wheel_separation>
+          <wheel_separation>${wheel_separation}</wheel_separation>
           <wheel_radius>0.075</wheel_radius>
           <max_linear_acceleration>1</max_linear_acceleration>
@@ -136,4 +136,55 @@
       </plugin>
     </gazebo>
+    <!-- Gazebo macro for Argo Wheels -->
+    <xacro:macro name="rox_argo_wheel_gazebo_macro" params="name">
+      <gazebo reference="${name}_link">
+        <mu1>0.001</mu1>
+        <mu2>0.001</mu2>
+        <kp>100000.0</kp>
+        <kd>1.0</kd>
+        <minDepth>0.000</minDepth>
+        <fdir1>1 0 0</fdir1>
+      </gazebo>
+    </xacro:macro>
+    <!-- Gazebo macro for Differential Castor Wheels -->
+    <xacro:macro name="rox_caster_wheel_gazebo_macro" params="name">
+      <gazebo reference="${name}_link">
+        <mu1>0.001</mu1>
+        <mu2>0.001</mu2>
+      </gazebo>
+    </xacro:macro>
+    <!-- Gazebo macro for Differential Wheels -->
+    <xacro:macro name="rox_diff_wheel_gazebo_macro" params="name">
+      <gazebo reference="${name}_link">
+        <mu1>1.0</mu1>
+        <mu2>1.0</mu2>
+        <kp>1000000.0</kp>
+        <kd>1.0</kd>
+        <minDepth>0.000</minDepth>
+        <fdir1>1 0 0</fdir1>
+      </gazebo>
+    </xacro:macro>
+    <!--Argo Drive-->
+    <xacro:if value="${rox_typ == 'argo'}">
+      <xacro:rox_argo_wheel_gazebo_macro name="wheel_front_left"/>
+      <xacro:rox_argo_wheel_gazebo_macro name="wheel_front_right"/>
+      <xacro:rox_argo_wheel_gazebo_macro name="wheel_back_left"/>
+      <xacro:rox_argo_wheel_gazebo_macro name="wheel_back_right"/>
+    </xacro:if>
+    <!--Diff Drive-->
+    <xacro:if value="${rox_typ == 'diff'}">
+      <xacro:rox_diff_wheel_gazebo_macro name="wheel_left"/>
+      <xacro:rox_diff_wheel_gazebo_macro name="wheel_right"/>
+      <xacro:rox_caster_wheel_gazebo_macro name="caster_wheel_front_left"/>
+      <xacro:rox_caster_wheel_gazebo_macro name="caster_wheel_front_right"/>
+      <xacro:rox_caster_wheel_gazebo_macro name="caster_wheel_back_left"/>
+      <xacro:rox_caster_wheel_gazebo_macro name="caster_wheel_back_right"/>
+    </xacro:if>
+    <!--Trike Drive-->
+    <xacro:if value="${rox_typ == 'trike'}">
+      <xacro:rox_diff_wheel_gazebo_macro name="wheel_left"/>
+      <xacro:rox_diff_wheel_gazebo_macro name="wheel_right"/>
+      <xacro:rox_caster_wheel_gazebo_macro name="caster_back"/>
+    </xacro:if>
   </xacro:macro>
 </robot>
