Commit message: Refactored launch files, fixed urdf indentations, changed outdated 'joint_properties' tag in urdf to 'dynamics', added initial_joint_controller condition in bringup_launch, removed meca drive and frame type

File: rox_description/urdf/rox.urdf.xacro (robot description, xacro)
@@ -1,142 +1,142 @@
 <?xml version="1.0" ?>
+<!--
+Author: Pradheep Padmanabhan
+Contributor: Adarsh Karan K P
+-->
 <robot xmlns:xacro="http://www.ros.org/wiki/xacro" name="rox">
-    <!-- Xacro Arguments-->
-    <xacro:arg name="frame_type" default="short"/>
-    <xacro:arg name="rox_type" default="argo"/>
-    <xacro:arg name="joint_type" default="fixed"/>
-    <xacro:arg name="scanner" default="nanoscan"/>
-    <xacro:arg name="arm_type" default=""/>
-    <xacro:arg name="use_gz" default="false"/>
-    <xacro:arg name="use_imu" default="false"/>
-    <xacro:arg name="use_d435" default="false"/>
-    <xacro:arg name="use_ur_dc" default="false"/>
-    <xacro:arg name="arm_parent" default="cabinet_link"/>
-    <xacro:arg name="force_abs_paths" default="false"/>
-    <xacro:arg name="simulation_controllers" default=""/>
-    <xacro:arg name="use_mock_hardware" default="false" />
-    <xacro:arg name="mock_sensor_commands" default="false" />
-    <!-- Xacro Properties -->
-    <xacro:property name="frame" value="$(arg frame_type)"/>
-    <xacro:property name="rox_typ" default="$(arg rox_type)"/>
-    <xacro:property name="joint_typ" value="$(arg joint_type)"/>
-    <xacro:property name="scanner_typ" value="$(arg scanner)"/>
-    <xacro:property name="arm" value="$(arg arm_type)"/>
-    <xacro:property name="gz" value="$(arg use_gz)"/>
-    <xacro:property name="use_arm" value="false"/>
-    <xacro:property name="imu" value="$(arg use_imu)"/>
-    <xacro:property name="d435" value="$(arg use_d435)"/>
-    <xacro:property name="ur_dc" value="$(arg use_ur_dc)"/>
-    <!-- Include xacro files -->
-    <xacro:include filename="$(find rox_description)/urdf/xacros/frame.xacro" />
-    <!-- Nanoscan -->
-    <xacro:include filename="$(find rox_description)/urdf/xacros/sick_nanoscan.xacro" />
-    <!-- PSenScan -->
-    <xacro:include filename="$(find rox_description)/urdf/xacros/pilz_psenscan.xacro" />
-    <!-- checking if one of the UR arms is used -->
-    <xacro:if value="${arm == 'ur5' or arm == 'ur10' or arm == 'ur5e' or arm == 'ur10e' or arm == 'ec66' or arm == 'cs66'}">
-        <xacro:property name="use_arm" value="true"/>
+<!-- This is the main URDF file for rox robot -->
+  <!-- Xacro Arguments-->
+  <xacro:arg name="rox_type" default="argo"/>
+  <xacro:arg name="joint_type" default="fixed"/>
+  <xacro:arg name="scanner" default="nanoscan"/>
+  <xacro:arg name="arm_type" default=""/>
+  <xacro:arg name="use_gz" default="false"/>
+  <xacro:arg name="use_imu" default="false"/>
+  <xacro:arg name="use_d435" default="false"/>
+  <xacro:arg name="use_ur_dc" default="false"/>
+  <xacro:arg name="arm_parent" default="cabinet_link"/>
+  <xacro:arg name="force_abs_paths" default="false"/>
+  <xacro:arg name="simulation_controllers" default=""/>
+  <xacro:arg name="use_mock_hardware" default="false" />
+  <xacro:arg name="mock_sensor_commands" default="false" />
+  <!-- Xacro Properties -->
+  <xacro:property name="rox_typ" default="$(arg rox_type)"/>
+  <xacro:property name="joint_typ" value="$(arg joint_type)"/>
+  <xacro:property name="scanner_typ" value="$(arg scanner)"/>
+  <xacro:property name="arm" value="$(arg arm_type)"/>
+  <xacro:property name="gz" value="$(arg use_gz)"/>
+  <xacro:property name="imu" value="$(arg use_imu)"/>
+  <xacro:property name="d435" value="$(arg use_d435)"/>
+  <xacro:property name="ur_dc" value="$(arg use_ur_dc)"/>
+  <!-- Include xacro files -->
+  <xacro:include filename="$(find rox_description)/urdf/xacros/frame.xacro" />
+  <!-- Nanoscan -->
+  <xacro:include filename="$(find rox_description)/urdf/xacros/sick_nanoscan.xacro" />
+  <!-- PSenScan -->
+  <xacro:include filename="$(find rox_description)/urdf/xacros/pilz_psenscan.xacro" />
+  <!-- Building the robot from here -->
+  <link name="base_link" />
+  <xacro:rox_base
+    name="base_footprint"
+    parent="base_link"
+    >
+    <origin xyz="0 0 0" rpy="0 0 0" />
+  </xacro:rox_base>
+  <!-- Argo drives -->
+  <xacro:if value="${rox_typ == 'argo'}">
+    <xacro:include filename="$(find rox_description)/urdf/xacros/argo_drive.xacro" />
+    <xacro:argo_drive parent="base_link"/>
+  </xacro:if>
+  <!-- Diff drive -->
+  <!-- Includes both Trike and Diff -->
+  <xacro:if value="${rox_typ == 'diff'}">
+    <xacro:include filename="$(find rox_description)/urdf/xacros/diff_drive.xacro" />
+    <xacro:property name="wheel_separation" value="0.634" />
+    <xacro:diff_drive parent="base_link" wheel_separation="${wheel_separation}"/>
+  </xacro:if>
+  <!-- Trike drive -->
+  <xacro:if value="${rox_typ == 'trike'}">
+    <xacro:include filename="$(find rox_description)/urdf/xacros/trike_drive.xacro" />
+    <xacro:property name="wheel_separation" value="0.5955" />
+    <xacro:trike_drive parent="base_link" wheel_separation="${wheel_separation}"/>
+  </xacro:if>
+  <!-- Laser scanners -->
+  <!-- Nanoscans -->
+  <xacro:if value="${scanner_typ == 'nanoscan'}">
+    <xacro:sick_nanoscan name="lidar_1" parent="base_link">
+      <origin rpy="${pi} 0 ${pi/4}" xyz="${0.2995} 0.269 0.189"/>
+    </xacro:sick_nanoscan>
+    <xacro:sick_nanoscan name="lidar_2" parent="base_link">
+      <origin rpy="${pi} 0 -${pi - pi/4}" xyz="-${0.2995} -0.269 0.189"/>
+    </xacro:sick_nanoscan>
+  </xacro:if>
+  <!-- Pilz -->
+  <xacro:if value="${scanner_typ == 'psenscan'}">
+    <xacro:pilz_psenscan name="lidar_1" parent="base_link">
+      <origin rpy="0 0 ${pi/4}" xyz="${0.3016} 0.2719 0.191"/>
+    </xacro:pilz_psenscan>
+    <xacro:pilz_psenscan name="lidar_2" parent="base_link">
+      <origin rpy="0 0 -${pi - pi/4}" xyz="-${0.3016} -0.2719 0.191"/>
+    </xacro:pilz_psenscan>
+  </xacro:if>
+  <!-- IMU -->
+  <xacro:if value="${imu == True}">
+    <link name="imu_link">
+      <inertial>
+        <mass value="0.001" />
+        <origin xyz="0 0 0" rpy="0 0 0" />
+        <inertia
+          ixx="0.0001"
+          ixy="0"
+          ixz="0"
+          iyy="0.000001"
+          iyz="0"
+          izz="0.0001"
+          />
+      </inertial>
+    </link>
+    <joint name="imu_joint" type="fixed">
+      <axis xyz="0 1 0"/>
+      <origin rpy="0 0 0" xyz="-0.052 0.208 0.266"/>
+      <parent link="base_link"/>
+      <child link="imu_link"/>
+    </joint>
+  </xacro:if>
+  <!-- Realsense D435 -->
+  <xacro:if value="${d435 == True}">
+    <xacro:include filename="$(find realsense2_description)/urdf/_d435.urdf.xacro"/>
+    <xacro:sensor_d435 parent="base_link">
+      <origin xyz="0.292 0.0 0.716" rpy="0 0 0"/>
+    </xacro:sensor_d435>
+  </xacro:if>
+  <!-- arm -->
+  <xacro:unless value="${arm == ''}">
+    <!-- Include cabinet -->
+    <xacro:include filename="$(find rox_description)/urdf/xacros/cabinet.xacro" />
+    <xacro:cabinet name="cabinet" parent="base_footprint">
+      <origin rpy="0 0 0" xyz="0 0 0.33"/>
+    </xacro:cabinet>
+    <!-- Universal Robotics (UR) Arms-->
+    <xacro:if value="${arm == 'ur5' or arm == 'ur10' or arm == 'ur5e' or arm == 'ur10e'}">
+      <!-- Different height for AC arm-->
+      <xacro:if value="${ur_dc == False}">
+        <xacro:property name="arm_height" value="0.376" />
+      </xacro:if>
+      <xacro:if value="${ur_dc == True}">
+        <xacro:property name="arm_height" value="0.276" />
+      </xacro:if>
+      <!-- Include the UR arm -->
+      <xacro:include filename="$(find rox_description)/urdf/xacros/ur_arm.urdf.xacro"/>
     </xacro:if>
-    <!-- Assigning Xacro properties -->
-    <xacro:if value="${frame == 'short'}">
-        <xacro:property name="frame_len" value="0.0" />
+    <!-- Elite Arms-->
+    <xacro:if value="${arm == 'ec66' or arm == 'cs66'}">
+      <xacro:property name="arm_height" value="0.376" />
+      <xacro:include filename="$(find rox_description)/urdf/xacros/elite_arm.urdf.xacro"/>
     </xacro:if>
-    <xacro:if value="${frame == 'long'}">
-        <xacro:property name="frame_len" value="0.13" />
-    </xacro:if>
-    <!-- Building the robot from here -->
-    <link name="base_link" />
-    <xacro:rox_base name="base_footprint"  parent="base_link"
-        type="${frame}">
-        <origin xyz="0 0 0" rpy="0 0 0" />
-    </xacro:rox_base>
-    <!-- Argo drives -->
-    <xacro:if value="${rox_typ == 'argo'}">
-        <xacro:include filename="$(find rox_description)/urdf/xacros/argo_drive.xacro" />
-        <xacro:argo_drive parent="base_link"/>
-    </xacro:if>
-    <!-- Diff drive -->
-    <!-- Includes both Trike and Diff -->
-    <xacro:if value="${rox_typ == 'diff'}">
-        <xacro:include filename="$(find rox_description)/urdf/xacros/diff_drive.xacro" />
-        <xacro:property name="wheel_separation" value="0.634" />
-        <xacro:diff_drive parent="base_link" wheel_separation="${wheel_separation}"/>
-    </xacro:if>
-    <!-- Trike drive -->
-    <xacro:if value="${rox_typ == 'trike'}">
-        <xacro:include filename="$(find rox_description)/urdf/xacros/trike_drive.xacro" />
-        <xacro:property name="wheel_separation" value="0.5955" />
-        <xacro:trike_drive parent="base_link" wheel_separation="${wheel_separation}"/>
-    </xacro:if>
-    <!-- Sensors -->
-    <!-- Laser scanners -->
-    <!-- Nanoscans -->
-    <xacro:if value="${scanner_typ == 'nanoscan'}">
-        <xacro:sick_nanoscan name="lidar_1" parent="base_link">
-            <origin rpy="${pi} 0 ${pi/4}" xyz="${0.2995 + frame_len} 0.269 0.189"/>
-        </xacro:sick_nanoscan>
-        <xacro:sick_nanoscan name="lidar_2" parent="base_link">
-            <origin rpy="${pi} 0 -${pi - pi/4}" xyz="-${0.2995 - frame_len} -0.269 0.189"/>
-        </xacro:sick_nanoscan>
-    </xacro:if>
-    <!-- Pilz -->
-    <xacro:if value="${scanner_typ == 'psenscan'}">
-        <xacro:pilz_psenscan name="lidar_1" parent="base_link">
-            <origin rpy="0 0 ${pi/4}" xyz="${0.3016 + frame_len} 0.2719 0.191"/>
-        </xacro:pilz_psenscan>
-        <xacro:pilz_psenscan name="lidar_2" parent="base_link">
-            <origin rpy="0 0 -${pi - pi/4}" xyz="-${0.3016 + frame_len} -0.2719 0.191"/>
-        </xacro:pilz_psenscan>
-    </xacro:if>
-    <!-- IMU -->
-    <xacro:if value="${imu == True}">
-        <link name="imu_link">
-            <inertial>
-                <mass value="0.001" />
-                <origin xyz="0 0 0" rpy="0 0 0" />
-                <inertia ixx="0.0001" ixy="0" ixz="0" iyy="0.000001" iyz="0" izz="0.0001" />
-            </inertial>
-        </link>
-        <joint name="imu_joint" type="fixed">
-            <axis xyz="0 1 0"/>
-            <origin rpy="0 0 0" xyz="-0.052 0.208 0.266"/>
-            <parent link="base_link"/>
-            <child link="imu_link"/>
-        </joint>
-    </xacro:if>
-    <!-- Realsense D435 -->
-    <xacro:if value="${d435 == True}">
-        <xacro:include filename="$(find realsense2_description)/urdf/_d435.urdf.xacro"/>
-        <xacro:sensor_d435 parent="base_link">
-            <origin xyz="0.292 0.0 0.716" rpy="0 0 0"/>
-        </xacro:sensor_d435>
-    </xacro:if>
-    <!-- arm -->
-    <xacro:if value="${use_arm}">
-        <!-- include cabinet -->
-        <xacro:include filename="$(find rox_description)/urdf/xacros/cabinet.xacro" />
-        <xacro:cabinet name="cabinet" parent="base_footprint">
-            <origin rpy="0 0 0" xyz="${frame_len} 0 0.33"/>
-        </xacro:cabinet>
-        <!-- Universal Robotics (UR) Arms-->
-        <xacro:if value="${arm == 'ur5' or arm == 'ur10' or arm == 'ur5e' or arm == 'ur10e'}">
-            <xacro:if value="${ur_dc == False}">
-                <!-- Different height for AC arm-->
-                <xacro:property name="arm_height" value="0.376" />
-            </xacro:if>
-            <xacro:if value="${ur_dc == True}">
-                <xacro:property name="arm_height" value="0.276" />
-            </xacro:if>
-            <xacro:include filename="$(find rox_description)/urdf/xacros/ur_arm.urdf.xacro"/>
-        </xacro:if>
-        <!-- Elite Arms-->
-        <xacro:if value="${arm == 'ec66' or arm == 'cs66'}">
-            <xacro:property name="arm_height" value="0.376" />
-            <xacro:include filename="$(find rox_description)/urdf/xacros/elite_arm.urdf.xacro"/>
-        </xacro:if>
-    </xacro:if>
-    <!-- Check if simulation needs to be used -->
-    <xacro:if value="${gz == True}">
-        <xacro:include filename="$(find rox_description)/urdf/xacros/gazebo.xacro" />
-        <xacro:gazebo_plugins />
-    </xacro:if>
+  </xacro:unless>
+  <!-- Check if simulation needs to be used -->
+  <xacro:if value="${gz == True}">
+    <xacro:include filename="$(find rox_description)/urdf/xacros/gazebo.xacro" />
+    <xacro:gazebo_plugins />
+  </xacro:if>
 </robot>

File: rox_description/urdf/xacros/argo_caster.xacro (robot description, xacro)
@@ -5,5 +5,5 @@
     <xacro:insert_block name="origin" />
     <axis xyz="1 0 0" />
-    <joint_properties damping="1." friction="1.0"/>
+    <dynamics damping="1." friction="1.0"/>
     <limit effort="1000.0" lower="-1e+16" upper="1e+16" velocity="100"/>
     <parent link="${parent}" />

File: rox_description/urdf/xacros/argo_drive.xacro (robot description, xacro)
@@ -7,20 +7,20 @@
         vis_rot="0 0 0" vis_pos="0 0 0"
         joint_type="${joint_typ}">
-        <origin rpy="0 0 ${pi}" xyz="${0.239 + frame_len} 0.229 0.123"/>
+        <origin rpy="0 0 ${pi}" xyz="${0.239} 0.229 0.123"/>
     </xacro:argo_caster>
     <xacro:argo_caster name="caster_front_right" parent="${parent}"
         vis_rot="0 0 ${pi}" vis_pos="0 0 0"
         joint_type="${joint_typ}">
-        <origin rpy="0 0 0" xyz="${0.239 + frame_len} -0.229 0.123"/>
+        <origin rpy="0 0 0" xyz="${0.239} -0.229 0.123"/>
     </xacro:argo_caster>
     <xacro:argo_caster name="caster_back_left" parent="${parent}"
         vis_rot="0 0 0" vis_pos="0 0 0"
         joint_type="${joint_typ}">
-        <origin rpy="0 0 ${pi}" xyz="-${0.239 + frame_len} 0.229 0.123"/>
+        <origin rpy="0 0 ${pi}" xyz="-${0.239} 0.229 0.123"/>
     </xacro:argo_caster>
     <xacro:argo_caster name="caster_back_right" parent="${parent}"
         vis_rot="0 0 ${pi}" vis_pos="0 0 0"
         joint_type="${joint_typ}">
-        <origin rpy="0 0 0" xyz="-${0.239 + frame_len} -0.229 0.123"/>
+        <origin rpy="0 0 0" xyz="-${0.239} -0.229 0.123"/>
     </xacro:argo_caster>
     <xacro:argo_wheel name="wheel_front_left" parent="caster_front_left_link"

File: rox_description/urdf/xacros/argo_wheel.xacro (robot description, xacro)
@@ -5,5 +5,5 @@
     <xacro:insert_block name="origin" />
     <limit effort="1000.0" lower="-1e+16" upper="1e+16" velocity="100"/>
-    <joint_properties damping="1.0" friction="1"/>
+    <dynamics damping="1.0" friction="1"/>
     <axis xyz="1 0 0" />
     <parent link="${parent}" />

File: rox_description/urdf/xacros/cabinet.xacro (robot description, xacro)
@@ -4,5 +4,5 @@
     <joint name="${name}_joint" type="fixed">
       <xacro:insert_block name="origin" />
-      <joint_properties damping="1" friction="1" />
+      <dynamics damping="1" friction="1" />
       <parent link="${parent}" />
       <child link="${name}_link" />

File: rox_description/urdf/xacros/diff_caster.xacro (robot description, xacro)
@@ -4,5 +4,5 @@
     <joint name="${name}_joint" type="${joint_type}">
       <xacro:insert_block name="origin" />
-      <joint_properties damping="1." friction="1.0"/>
+      <dynamics damping="1." friction="1.0"/>
       <limit effort="1000.0" lower="-1e+16" upper="1e+16" velocity="100"/>
       <axis xyz="1 0 0" />

File: rox_description/urdf/xacros/diff_drive.xacro (robot description, xacro)
@@ -7,5 +7,5 @@
         vis_rot="-${pi/2} 0 ${pi/2}" vis_pos="0 0 0" collision_pos="0.045 0 0"
         joint_type="fixed">
-        <origin rpy="0 0 0" xyz="${0.2045 + frame_len + 0.045} -0.220 0.124"/>
+        <origin rpy="0 0 0" xyz="${0.2045 + 0.045} -0.220 0.124"/>
         <!-- For the caster position 0.2785 is L3.2 and 0.045 is the Swivel lead -->
     </xacro:diff_caster>
@@ -13,5 +13,5 @@
         vis_rot="-${pi/2} 0 ${pi/2}" vis_pos="0 0 0" collision_pos="0.045 0 0"
         joint_type="fixed">
-        <origin rpy="0 0 0" xyz="${0.2045 + frame_len + 0.045} 0.220 0.124"/>
+        <origin rpy="0 0 0" xyz="${0.2045 + 0.045} 0.220 0.124"/>
         <!-- For the caster position 0.2785 is L3.2 and 0.045 is the Swivel lead -->
     </xacro:diff_caster>
@@ -19,5 +19,5 @@
         vis_rot="-${pi/2} 0 ${pi/2}" vis_pos="0 0 0" collision_pos="0.045 0 0"
         joint_type="fixed">
-        <origin rpy="0 0 0" xyz="-${0.2945 + frame_len - 0.045} -0.220 0.124"/>
+        <origin rpy="0 0 0" xyz="-${0.2945 - 0.045} -0.220 0.124"/>
         <!-- For the caster position 0.1885 is L3.2 and 0.045 is the Swivel lead -->
     </xacro:diff_caster>
@@ -25,5 +25,5 @@
         vis_rot="-${pi/2} 0 ${pi/2}" vis_pos="0 0 0" collision_pos="0.045 0 0"
         joint_type="fixed">
-        <origin rpy="0 0 0" xyz="-${0.2945 + frame_len - 0.045} 0.220 0.124"/>
+        <origin rpy="0 0 0" xyz="-${0.2945 - 0.045} 0.220 0.124"/>
         <!-- For the caster position 0.1885 is L3.2 and 0.045 is the Swivel lead -->
     </xacro:diff_caster>

File: rox_description/urdf/xacros/diff_wheel.xacro (robot description, xacro)
@@ -4,6 +4,6 @@
     <joint name="${name}_joint" type="${joint_type}">
       <xacro:insert_block name="origin" />
-    <limit effort="1000.0" lower="-1e+16" upper="1e+16" velocity="100"/>
-    <joint_properties damping="1.0" friction="1"/>
+      <limit effort="1000.0" lower="-1e+16" upper="1e+16" velocity="100"/>
+      <dynamics damping="1.0" friction="1"/>
       <axis xyz="0 1 0" />
       <parent link="${parent}" />
@@ -15,5 +15,5 @@
         <mass value="5.0" />
         <origin xyz="0 0 0" rpy="0 0 0" />
-<inertia ixx="0.02888" ixy="0" ixz="0" iyy="0.02888" iyz="0" izz="0.05625" />      </inertial>
+        <inertia ixx="0.02888" ixy="0" ixz="0" iyy="0.02888" iyz="0" izz="0.05625" />      </inertial>
       <visual>
         <origin rpy="${pi/2} 0 0" xyz="0 0 0" />

File: rox_description/urdf/xacros/frame.xacro (robot description, xacro)
@@ -1,5 +1,5 @@
 <?xml version="1.0"?>
 <robot xmlns:xacro="http://www.ros.org/wiki/xacro" name="rox">
-  <xacro:macro name="rox_base" params="name parent type *origin">
+  <xacro:macro name="rox_base" params="name parent *origin">
    <joint name="${name}_joint" type="fixed">
     <xacro:insert_block name="origin" />
@@ -18,5 +18,5 @@
         <origin xyz="0.0 0.0 0.0" rpy="0 0 0" />
         <geometry>
-          <mesh filename="package://rox_description/meshes/${type}_frame.dae" scale="0.1 0.1 0.1"/>
+          <mesh filename="package://rox_description/meshes/short_frame.dae" scale="0.1 0.1 0.1"/>
         </geometry>
       </visual>
@@ -24,5 +24,5 @@
         <origin xyz="0.0 0.0 0.0" rpy="0 0 0"/>
         <geometry>
-          <mesh filename="package://rox_description/meshes/${type}_frame.dae" scale="0.1 0.1 0.1"/>
+          <mesh filename="package://rox_description/meshes/short_frame.dae" scale="0.1 0.1 0.1"/>
         </geometry>
       </collision>

File: rox_description/urdf/xacros/trike_drive.xacro (robot description, xacro)
@@ -7,5 +7,5 @@
         vis_rot="-${pi/2} 0 -${pi/2}" vis_pos="0 0 0" collision_pos="-0.045 0 0"
         joint_type="fixed">
-        <origin rpy="0 0 0" xyz="-${0.2785 - 0.045 + frame_len} 0.0 0.124"/>
+        <origin rpy="0 0 0" xyz="-${0.2785 - 0.045} 0.0 0.124"/>
         <!-- For the caster position 0.2785 is L3.2 and 0.045 is the Swivel lead -->
     </xacro:diff_caster>
