Commit message: Added support for robotiq grippers (#65)
* Added support for robotiq grippers,updated urdf and launch files, fixed formatting

* removed d435 support from bringup launch file

* updated arm initial position to avoid collision with gripper

File: rox_description/urdf/rox.urdf.xacro (robot description, xacro)
@@ -7,26 +7,32 @@
 <!-- This is the main URDF file for rox robot -->
   <!-- Xacro Arguments-->
-  <xacro:arg name="rox_type" default="argo"/>
-  <xacro:arg name="joint_type" default="fixed"/>
-  <xacro:arg name="scanner" default="nanoscan"/>
-  <xacro:arg name="arm_type" default=""/>
   <xacro:arg name="use_gz" default="false"/>
   <xacro:arg name="use_imu" default="false"/>
   <xacro:arg name="use_d435" default="false"/>
+  <xacro:arg name="scanner_type" default="nanoscan"/>
+  <xacro:arg name="rox_type" default="argo"/>
+  <xacro:arg name="joint_type" default="fixed"/>
+  <!-- Manipulator Arguments-->
+  <xacro:arg name="arm_type" default=""/>
+  <xacro:arg name="arm_parent" default="cabinet_link"/>
+  <xacro:arg name="gripper_type" default=""/>
   <xacro:arg name="use_ur_dc" default="false"/>
-  <xacro:arg name="arm_parent" default="cabinet_link"/>
   <xacro:arg name="force_abs_paths" default="false"/>
   <xacro:arg name="simulation_controllers" default=""/>
   <xacro:arg name="use_mock_hardware" default="false" />
   <xacro:arg name="mock_sensor_commands" default="false" />
+  <xacro:arg name="include_arm_ros2_control" default="false"/>
+  <xacro:arg name="include_gripper_ros2_control" default="false"/>
   <!-- Xacro Properties -->
-  <xacro:property name="rox_typ" default="$(arg rox_type)"/>
-  <xacro:property name="joint_typ" value="$(arg joint_type)"/>
-  <xacro:property name="scanner_typ" value="$(arg scanner)"/>
-  <xacro:property name="arm" value="$(arg arm_type)"/>
   <xacro:property name="gz" value="$(arg use_gz)"/>
   <xacro:property name="imu" value="$(arg use_imu)"/>
   <xacro:property name="d435" value="$(arg use_d435)"/>
+  <xacro:property name="scanner" value="$(arg scanner_type)"/>
+  <xacro:property name="rox_typ" value="$(arg rox_type)"/>
+  <xacro:property name="joint_typ" value="$(arg joint_type)"/>
+  <xacro:property name="arm" value="$(arg arm_type)"/>
   <xacro:property name="ur_dc" value="$(arg use_ur_dc)"/>
+  <xacro:property name="gripper" value="$(arg gripper_type)"/>
+  <xacro:property name="use_mock" value="$(arg use_mock_hardware)"/>
   <!-- Include xacro files -->
   <xacro:include filename="$(find rox_description)/urdf/xacros/frame.xacro" />
@@ -67,5 +73,5 @@
   <!-- Laser scanners -->
   <!-- Nanoscans -->
-  <xacro:if value="${scanner_typ == 'nanoscan'}">
+  <xacro:if value="${scanner == 'nanoscan'}">
     <xacro:sick_nanoscan name="lidar_1" parent="base_link">
       <origin rpy="${pi} 0 ${pi/4}" xyz="${0.2995} 0.269 0.189"/>
@@ -76,5 +82,5 @@
   </xacro:if>
   <!-- Pilz -->
-  <xacro:if value="${scanner_typ == 'psenscan'}">
+  <xacro:if value="${scanner == 'psenscan'}">
     <xacro:pilz_psenscan name="lidar_1" parent="base_link">
       <origin rpy="0 0 ${pi/4}" xyz="${0.3016} 0.2719 0.191"/>
@@ -138,4 +144,36 @@
       <xacro:include filename="$(find rox_description)/urdf/xacros/elite_arm.urdf.xacro"/>
     </xacro:if>
+    <!-- add gripper-->
+    <xacro:unless value="${gripper == ''}">
+      <!-- ur_adapter for gripper-->
+      <xacro:if value="${gripper == '2f_140' or gripper == '2f_85'}">
+        <xacro:include filename="$(find robotiq_description)/urdf/ur_to_robotiq_adapter.urdf.xacro"/>
+        <xacro:ur_to_robotiq
+          prefix=""
+          parent="$(arg tf_prefix)tool0"
+          child="neo_gripper_mount_link"
+          rotation="${pi/2}"
+          />
+        <xacro:include filename="$(find robotiq_description)/urdf/robotiq_${gripper}_macro.urdf.xacro"/>
+        <xacro:robotiq_gripper name="robotiq_gripper"
+          prefix=""
+          parent="neo_gripper_mount_link"
+          use_mock_hardware="${use_mock}"
+          mock_sensor_commands="${use_mock}"
+          sim_gazebo="${gz}"
+          include_ros2_control="$(arg include_gripper_ros2_control)"
+          >
+          <origin xyz="0 0 0" rpy="0 0 -${pi / 2}"/>
+        </xacro:robotiq_gripper>
+      </xacro:if>
+      <xacro:if value="${gripper == 'epick'}">
+        <xacro:include filename="$(find epick_description)/urdf/epick_single_suction_cup.xacro"/>
+        <xacro:epick_single_suction_cup parent="$(arg tf_prefix)tool0"
+          use_fake_hardware="${use_mock}"
+          origin_xyz="0 0 0"
+          origin_rpy="0 0 -${pi / 2}"
+          />
+      </xacro:if>
+    </xacro:unless>
   </xacro:unless>
   <!-- Check if simulation needs to be used -->

File: rox_description/urdf/xacros/elite_arm.urdf.xacro (robot description, xacro)
@@ -55,5 +55,3 @@
       />
   </xacro:if>
-  <!-- include robotiq gripper-->
-  <!-- <xacro:include filename="$(find neo_simulation2)/components/arm/robotiq_gripper.urdf.xacro"/> -->
 </robot>

File: rox_description/urdf/xacros/ur_arm.urdf.xacro (robot description, xacro)
@@ -11,4 +11,5 @@
   <!-- Set use_gz = true for simulation -->
   <xacro:arg name="use_gz" default="false"/>
+  <xacro:arg name="include_arm_ros2_control" default="false"/>
   <!-- arm parameters -->
   <xacro:arg name="arm_type" default="ur10"/>
@@ -53,55 +54,57 @@
   <!-- this condition is to ensure that ros2_control doesn't interfere with gz_ros2_control during simulation  -->
   <xacro:unless value="$(arg use_gz)">
-    <!-- ros2_control related parameters -->
-    <xacro:arg name="headless_mode" default="false" />
-    <xacro:arg name="robot_ip" default="192.168.1.102" />
-    <xacro:arg name="script_filename" default="$(find ur_client_library)/resources/external_control.urscript"/>
-    <xacro:arg name="output_recipe_filename" default="$(find ur_robot_driver)/resources/rtde_output_recipe.txt"/>
-    <xacro:arg name="input_recipe_filename" default="$(find ur_robot_driver)/resources/rtde_input_recipe.txt"/>
-    <xacro:arg name="reverse_ip" default="0.0.0.0"/>
-    <xacro:arg name="script_command_port" default="50004"/>
-    <xacro:arg name="reverse_port" default="50001"/>
-    <xacro:arg name="script_sender_port" default="50002"/>
-    <xacro:arg name="trajectory_port" default="50003"/>
-    <!-- tool communication related parameters-->
-    <xacro:arg name="use_tool_communication" default="false" />
-    <xacro:arg name="tool_voltage" default="0" />
-    <xacro:arg name="tool_parity" default="0" />
-    <xacro:arg name="tool_baud_rate" default="115200" />
-    <xacro:arg name="tool_stop_bits" default="1" />
-    <xacro:arg name="tool_rx_idle_chars" default="1.5" />
-    <xacro:arg name="tool_tx_idle_chars" default="3.5" />
-    <xacro:arg name="tool_device_name" default="/tmp/ttyUR" />
-    <xacro:arg name="tool_tcp_port" default="54321" />
-    <xacro:arg name="use_mock_hardware" default="false" />
-    <xacro:arg name="mock_sensor_commands" default="false" />
-    <xacro:ur_ros2_control
-      name="$(arg arm_type)"
-      tf_prefix="$(arg tf_prefix)"
-      kinematics_parameters_file="$(arg kinematics_params)"
-      transmission_hw_interface="$(arg transmission_hw_interface)"
-      headless_mode="$(arg headless_mode)"
-      initial_positions="${ur_initial_positions}"
-      use_tool_communication="$(arg use_tool_communication)"
-      tool_voltage="$(arg tool_voltage)"
-      tool_parity="$(arg tool_parity)"
-      tool_baud_rate="$(arg tool_baud_rate)"
-      tool_stop_bits="$(arg tool_stop_bits)"
-      tool_rx_idle_chars="$(arg tool_rx_idle_chars)"
-      tool_tx_idle_chars="$(arg tool_tx_idle_chars)"
-      tool_device_name="$(arg tool_device_name)"
-      tool_tcp_port="$(arg tool_tcp_port)"
-      robot_ip="$(arg robot_ip)"
-      script_filename="$(arg script_filename)"
-      output_recipe_filename="$(arg output_recipe_filename)"
-      input_recipe_filename="$(arg input_recipe_filename)"
-      reverse_ip="$(arg reverse_ip)"
-      script_command_port="$(arg script_command_port)"
-      reverse_port="$(arg reverse_port)"
-      script_sender_port="$(arg script_sender_port)"
-      trajectory_port="$(arg trajectory_port)"
-      use_mock_hardware="$(arg use_mock_hardware)"
-      mock_sensor_commands="$(arg mock_sensor_commands)"
-      />
+    <xacro:if value="$(arg include_arm_ros2_control)">
+      <!-- ros2_control related parameters -->
+      <xacro:arg name="headless_mode" default="false" />
+      <xacro:arg name="robot_ip" default="192.168.1.102" />
+      <xacro:arg name="script_filename" default="$(find ur_client_library)/resources/external_control.urscript"/>
+      <xacro:arg name="output_recipe_filename" default="$(find ur_robot_driver)/resources/rtde_output_recipe.txt"/>
+      <xacro:arg name="input_recipe_filename" default="$(find ur_robot_driver)/resources/rtde_input_recipe.txt"/>
+      <xacro:arg name="reverse_ip" default="0.0.0.0"/>
+      <xacro:arg name="script_command_port" default="50004"/>
+      <xacro:arg name="reverse_port" default="50001"/>
+      <xacro:arg name="script_sender_port" default="50002"/>
+      <xacro:arg name="trajectory_port" default="50003"/>
+      <!-- tool communication related parameters-->
+      <xacro:arg name="use_tool_communication" default="false" />
+      <xacro:arg name="tool_voltage" default="0" />
+      <xacro:arg name="tool_parity" default="0" />
+      <xacro:arg name="tool_baud_rate" default="115200" />
+      <xacro:arg name="tool_stop_bits" default="1" />
+      <xacro:arg name="tool_rx_idle_chars" default="1.5" />
+      <xacro:arg name="tool_tx_idle_chars" default="3.5" />
+      <xacro:arg name="tool_device_name" default="/tmp/ttyUR" />
+      <xacro:arg name="tool_tcp_port" default="54321" />
+      <xacro:arg name="use_mock_hardware" default="false" />
+      <xacro:arg name="mock_sensor_commands" default="false" />
+      <xacro:ur_ros2_control
+        name="$(arg arm_type)"
+        tf_prefix="$(arg tf_prefix)"
+        kinematics_parameters_file="$(arg kinematics_params)"
+        transmission_hw_interface="$(arg transmission_hw_interface)"
+        headless_mode="$(arg headless_mode)"
+        initial_positions="${ur_initial_positions}"
+        use_tool_communication="$(arg use_tool_communication)"
+        tool_voltage="$(arg tool_voltage)"
+        tool_parity="$(arg tool_parity)"
+        tool_baud_rate="$(arg tool_baud_rate)"
+        tool_stop_bits="$(arg tool_stop_bits)"
+        tool_rx_idle_chars="$(arg tool_rx_idle_chars)"
+        tool_tx_idle_chars="$(arg tool_tx_idle_chars)"
+        tool_device_name="$(arg tool_device_name)"
+        tool_tcp_port="$(arg tool_tcp_port)"
+        robot_ip="$(arg robot_ip)"
+        script_filename="$(arg script_filename)"
+        output_recipe_filename="$(arg output_recipe_filename)"
+        input_recipe_filename="$(arg input_recipe_filename)"
+        reverse_ip="$(arg reverse_ip)"
+        script_command_port="$(arg script_command_port)"
+        reverse_port="$(arg reverse_port)"
+        script_sender_port="$(arg script_sender_port)"
+        trajectory_port="$(arg trajectory_port)"
+        use_mock_hardware="$(arg use_mock_hardware)"
+        mock_sensor_commands="$(arg mock_sensor_commands)"
+        />
+    </xacro:if>
   </xacro:unless>
   <!-- If gz simulation is used -->
@@ -126,5 +129,3 @@
       />
   </xacro:if>
-  <!-- include robotiq gripper-->
-  <!-- <xacro:include filename="$(find neo_simulation2)/components/arm/robotiq_gripper.urdf.xacro"/> -->
 </robot>
